File: KiCad/BeanBike/Controller/Controller.kicad_sch (KiCad schematic)
At the start: 0 parts

Commit message: Power Circuit V1
Other:
- sheet Controller renamed MCU
Changed lines of the file:
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@@
 			(color 0 0 0 0.0000)
 		)
-		(property "Sheetname" "Controller"
+		(property "Sheetname" "MCU"
 			(at 160.02 14.5284 0)
 			(effects

Commit message: Connectors
Other:
- added sheet Connectors (beanbike_controller_connectors.kicad_sch)
Changed lines of the file:
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@@
+	)
+	(sheet
+		(at 160.02 102.87)
+		(size 119.38 57.15)
+		(exclude_from_sim no)
+		(in_bom yes)
+		(on_board yes)
+		(dnp no)
+		(fields_autoplaced yes)
+		(stroke
+			(width 0.1524)
+			(type solid)
+		)
+		(fill
+			(color 0 0 0 0.0000)
+		)
+		(property "Sheetname" "Connectors"
+			(at 160.02 102.1584 0)
+			(effects
+				(font
+					(size 1.27 1.27)
+				)
+				(justify left bottom)
+			)
+		)
+		(property "Sheetfile" "beanbike_controller_connectors.kicad_sch"
+			(at 160.02 160.6046 0)
+			(effects
+				(font
+					(size 1.27 1.27)
+				)
+				(justify left top)
+			)
+		)
+		(instances
+			(project "Controller"
+				(path "/645e8d68-d9e1-48b3-98a5-3b81aa58d1ea"
+					(page "4")
+				)
+			)
+		)
 	)
 	(sheet

Commit message: PCB v1
Whole lotta stuff
Other:
- added sheet Motor (beanbike_controller_motor.kicad_sch)
Changed lines of the file:
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@@
+	)
+	(sheet
+		(at 15.24 102.87)
+		(size 93.98 57.15)
+		(exclude_from_sim no)
+		(in_bom yes)
+		(on_board yes)
+		(dnp no)
+		(fields_autoplaced yes)
+		(stroke
+			(width 0.1524)
+			(type solid)
+		)
+		(fill
+			(color 0 0 0 0.0000)
+		)
+		(property "Sheetname" "Motor"
+			(at 15.24 102.1584 0)
+			(effects
+				(font
+					(size 1.27 1.27)
+				)
+				(justify left bottom)
+			)
+		)
+		(property "Sheetfile" "beanbike_controller_motor.kicad_sch"
+			(at 15.24 160.6046 0)
+			(effects
+				(font
+					(size 1.27 1.27)
+				)
+				(justify left top)
+			)
+		)
+		(instances
+			(project "Controller"
+				(path "/645e8d68-d9e1-48b3-98a5-3b81aa58d1ea"
+					(page "5")
+				)
+			)
+		)
 	)
 	(sheet
