File: KiCad/BeanBike/Controller/beanbike_controller_12v.kicad_sch (KiCad schematic)
At the start: 11 parts

Commit message: PCB v2
Connections:
- net 24v: now also C14.1
- net GND: now also C13.2
Other:
- moved on the sheet: C13, C14
Changed lines of the file:
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@@
+	)
+	(junction
+		(at 88.9 93.98)
+		(diameter 0)
+		(color 0 0 0 0)
 	)
 	(junction
@@
 	)
 	(junction
+		(at 88.9 109.22)
+		(diameter 0)
+		(color 0 0 0 0)
+	)
+	(junction
 		(at 168.91 95.25)
 		(diameter 0)
@@
 	)
 	(junction
+		(at 81.28 109.22)
+		(diameter 0)
+		(color 0 0 0 0)
+	)
+	(junction
 		(at 95.25 93.98)
 		(diameter 0)
@@
 	)
 	(junction
-		(at 81.28 109.22)
-		(diameter 0)
-		(color 0 0 0 0)
-	)
-	(junction
 		(at 142.24 124.46)
 		(diameter 0)
@@
 	(wire
 		(pts
-			(xy 81.28 109.22) (xy 95.25 109.22)
+			(xy 81.28 109.22) (xy 88.9 109.22)
 		)
 		(stroke
@@
 	(wire
 		(pts
-			(xy 81.28 93.98) (xy 95.25 93.98)
+			(xy 81.28 93.98) (xy 88.9 93.98)
 		)
 		(stroke
@@
 	(wire
 		(pts
+			(xy 81.28 97.79) (xy 81.28 93.98)
+		)
+		(stroke
+			(width 0)
+			(type default)
+		)
+	)
+	(wire
+		(pts
 			(xy 215.9 102.87) (xy 215.9 105.41)
 		)
@@
 	(wire
 		(pts
+			(xy 88.9 93.98) (xy 88.9 97.79)
+		)
+		(stroke
+			(width 0)
+			(type default)
+		)
+	)
+	(wire
+		(pts
 			(xy 172.72 95.25) (xy 172.72 100.33)
 		)
@@
 	(wire
 		(pts
+			(xy 81.28 105.41) (xy 81.28 109.22)
+		)
+		(stroke
+			(width 0)
+			(type default)
+		)
+	)
+	(wire
+		(pts
 			(xy 124.46 95.25) (xy 114.3 95.25)
 		)
@@
 	(wire
 		(pts
+			(xy 88.9 109.22) (xy 95.25 109.22)
+		)
+		(stroke
+			(width 0)
+			(type default)
+		)
+	)
+	(wire
+		(pts
 			(xy 142.24 120.65) (xy 142.24 124.46)
 		)
@@
 		(pts
 			(xy 191.77 124.46) (xy 171.45 124.46)
+		)
+		(stroke
+			(width 0)
+			(type default)
+		)
+	)
+	(wire
+		(pts
+			(xy 88.9 93.98) (xy 95.25 93.98)
+		)
+		(stroke
+			(width 0)
+			(type default)
+		)
+	)
+	(wire
+		(pts
+			(xy 88.9 105.41) (xy 88.9 109.22)
 		)
 		(stroke
@@
 	(symbol
 		(lib_id "Device:C")
-		(at 81.28 105.41 0)
+		(at 88.9 101.6 0)
 		(unit 1)
 		(exclude_from_sim no)
@@
 		(fields_autoplaced yes)
 		(property "Reference" "C14"
-			(at 85.09 104.1399 0)
+			(at 92.71 100.3299 0)
 			(effects
 				(font
@@
 		)
 		(property "Value" "2.2uF"
-			(at 85.09 106.6799 0)
+			(at 92.71 102.8699 0)
 			(effects
 				(font
@@
 		)
 		(property "Footprint" "Capacitor_SMD:C_0201_0603Metric"
-			(at 82.2452 109.22 0)
+			(at 89.8652 105.41 0)
 			(effects
 				(font
@@
 		)
 		(property "Datasheet" "~"
-			(at 81.28 105.41 0)
+			(at 88.9 101.6 0)
 			(effects
 				(font
@@
 		)
 		(property "Description" "Unpolarized capacitor"
-			(at 81.28 105.41 0)
+			(at 88.9 101.6 0)
 			(effects
 				(font
@@
 	(symbol
 		(lib_id "Device:C")
-		(at 81.28 97.79 0)
+		(at 81.28 101.6 0)
 		(unit 1)
 		(exclude_from_sim no)
@@
 		(fields_autoplaced yes)
 		(property "Reference" "C13"
-			(at 85.09 96.5199 0)
+			(at 85.09 100.3299 0)
 			(effects
 				(font
@@
 		)
 		(property "Value" "2.2uF"
-			(at 85.09 99.0599 0)
+			(at 85.09 102.8699 0)
 			(effects
 				(font
@@
 		)
 		(property "Footprint" "Capacitor_SMD:C_0201_0603Metric"
-			(at 82.2452 101.6 0)
+			(at 82.2452 105.41 0)
 			(effects
 				(font
@@
 		)
 		(property "Datasheet" "~"
-			(at 81.28 97.79 0)
+			(at 81.28 101.6 0)
 			(effects
 				(font
@@
 		)
 		(property "Description" "Unpolarized capacitor"
-			(at 81.28 97.79 0)
-			(effects
-				(font
+			(at 81.28 101.6 0)
+			(effects
+				(font
