File: KiCad/BeanBike/Controller/beanbike_controller_24v.kicad_sch (KiCad schematic)
At the start: 12 parts

Commit message: PCB v2
Connections:
- net 48V: now also C8.1
- net GND: now also C7.2
Other:
- moved on the sheet: C7, C8
Changed lines of the file:
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@@
+	)
+	(junction
+		(at 77.47 109.22)
+		(diameter 0)
+		(color 0 0 0 0)
 	)
 	(junction
@@
 	)
 	(junction
+		(at 87.63 93.98)
+		(diameter 0)
+		(color 0 0 0 0)
+	)
+	(junction
 		(at 95.25 93.98)
 		(diameter 0)
@@
 	)
 	(junction
-		(at 81.28 93.98)
-		(diameter 0)
-		(color 0 0 0 0)
-	)
-	(junction
 		(at 114.3 97.79)
 		(diameter 0)
@@
 	)
 	(junction
-		(at 81.28 109.22)
-		(diameter 0)
-		(color 0 0 0 0)
-	)
-	(junction
 		(at 142.24 124.46)
 		(diameter 0)
@@
 	)
 	(junction
+		(at 87.63 109.22)
+		(diameter 0)
+		(color 0 0 0 0)
+	)
+	(junction
+		(at 77.47 93.98)
+		(diameter 0)
+		(color 0 0 0 0)
+	)
+	(junction
 		(at 171.45 124.46)
 		(diameter 0)
@@
 	(wire
 		(pts
-			(xy 71.12 109.22) (xy 81.28 109.22)
-		)
-		(stroke
-			(width 0)
-			(type default)
-		)
-	)
-	(wire
-		(pts
-			(xy 73.66 93.98) (xy 81.28 93.98)
+			(xy 77.47 109.22) (xy 87.63 109.22)
+		)
+		(stroke
+			(width 0)
+			(type default)
+		)
+	)
+	(wire
+		(pts
+			(xy 77.47 105.41) (xy 77.47 109.22)
+		)
+		(stroke
+			(width 0)
+			(type default)
+		)
+	)
+	(wire
+		(pts
+			(xy 71.12 109.22) (xy 77.47 109.22)
+		)
+		(stroke
+			(width 0)
+			(type default)
+		)
+	)
+	(wire
+		(pts
+			(xy 73.66 93.98) (xy 77.47 93.98)
 		)
 		(stroke
@@
 	(wire
 		(pts
-			(xy 81.28 109.22) (xy 95.25 109.22)
-		)
-		(stroke
-			(width 0)
-			(type default)
-		)
-	)
-	(wire
-		(pts
 			(xy 105.41 93.98) (xy 105.41 100.33)
 		)
@@
 	(wire
 		(pts
+			(xy 77.47 93.98) (xy 77.47 97.79)
+		)
+		(stroke
+			(width 0)
+			(type default)
+		)
+	)
+	(wire
+		(pts
 			(xy 105.41 107.95) (xy 105.41 105.41)
 		)
@@
 	(wire
 		(pts
-			(xy 81.28 93.98) (xy 95.25 93.98)
-		)
-		(stroke
-			(width 0)
-			(type default)
-		)
-	)
-	(wire
-		(pts
 			(xy 160.02 107.95) (xy 171.45 107.95)
 		)
@@
 	(wire
 		(pts
+			(xy 87.63 109.22) (xy 95.25 109.22)
+		)
+		(stroke
+			(width 0)
+			(type default)
+		)
+	)
+	(wire
+		(pts
+			(xy 87.63 93.98) (xy 87.63 97.79)
+		)
+		(stroke
+			(width 0)
+			(type default)
+		)
+	)
+	(wire
+		(pts
+			(xy 77.47 93.98) (xy 87.63 93.98)
+		)
+		(stroke
+			(width 0)
+			(type default)
+		)
+	)
+	(wire
+		(pts
+			(xy 87.63 105.41) (xy 87.63 109.22)
+		)
+		(stroke
+			(width 0)
+			(type default)
+		)
+	)
+	(wire
+		(pts
 			(xy 237.49 95.25) (xy 215.9 95.25)
 		)
@@
 		(pts
 			(xy 95.25 93.98) (xy 105.41 93.98)
+		)
+		(stroke
+			(width 0)
+			(type default)
+		)
+	)
+	(wire
+		(pts
+			(xy 87.63 93.98) (xy 95.25 93.98)
 		)
 		(stroke
@@
 	(symbol
 		(lib_id "Device:C")
-		(at 81.28 97.79 0)
+		(at 77.47 101.6 0)
 		(unit 1)
 		(exclude_from_sim no)
@@
 		(fields_autoplaced yes)
 		(property "Reference" "C7"
-			(at 85.09 96.5199 0)
+			(at 81.28 100.3299 0)
 			(effects
 				(font
@@
 		)
 		(property "Value" "2.2uF"
-			(at 85.09 99.0599 0)
+			(at 81.28 102.8699 0)
 			(effects
 				(font
@@
 		)
 		(property "Footprint" "Capacitor_SMD:C_0201_0603Metric"
-			(at 82.2452 101.6 0)
+			(at 78.4352 105.41 0)
 			(effects
 				(font
@@
 		)
 		(property "Datasheet" "~"
-			(at 81.28 97.79 0)
+			(at 77.47 101.6 0)
 			(effects
 				(font
@@
 		)
 		(property "Description" "Unpolarized capacitor"
-			(at 81.28 97.79 0)
+			(at 77.47 101.6 0)
 			(effects
 				(font
@@
 	(symbol
 		(lib_id "Device:C")
-		(at 81.28 105.41 0)
+		(at 87.63 101.6 0)
 		(unit 1)
 		(exclude_from_sim no)
@@
 		(fields_autoplaced yes)
 		(property "Reference" "C8"
-			(at 85.09 104.1399 0)
+			(at 91.44 100.3299 0)
 			(effects
 				(font
@@
 		)
 		(property "Value" "2.2uF"
-			(at 85.09 106.6799 0)
+			(at 91.44 102.8699 0)
 			(effects
 				(font
@@
 		)
 		(property "Footprint" "Capacitor_SMD:C_0201_0603Metric"
-			(at 82.2452 109.22 0)
+			(at 88.5952 105.41 0)
 			(effects
 				(font
@@
 		)
 		(property "Datasheet" "~"
-			(at 81.28 105.41 0)
+			(at 87.63 101.6 0)
 			(effects
 				(font
@@
 		)
 		(property "Description" "Unpolarized capacitor"
-			(at 81.28 105.41 0)
-			(effects
-				(font
+			(at 87.63 101.6 0)
+			(effects
+				(font
