File: KiCad/BeanBike/Controller/beanbike_power.kicad_sch (KiCad schematic)
At the start: 0 parts

Commit message: Power Circuit V1
Parts:
- added F1: Fuse, symbol Device:Fuse
- added J1: XT80 Male, symbol Connector:Conn_01x02_Pin
- added R1: 180k, symbol Device:R
- added R2: 10k, symbol Device:R
- added SW1: SW_Push, symbol Switch:SW_Push
- added U2: JTD2048S3V3, Converter_DCDC:Converter_DCDC_XP_POWER_JTDxxxxxxx_THT, symbol Converter_DCDC:JTD2048S3V3
- added U3: JTD2048S05, Converter_DCDC:Converter_DCDC_XP_POWER_JTDxxxxxxx_THT, symbol Converter_DCDC:JTD2048S05
- added U4: JTD2048S12, Converter_DCDC:Converter_DCDC_XP_POWER_JTDxxxxxxx_THT, symbol Converter_DCDC:JTD2048S12
Connections:
- new net: F1.2, SW1.1
- new net +12V: U4.3 (+VOUT)
- new net +3.3V: U2.3 (+VOUT)
- new net +5V: U3.3 (+VOUT)
- new net +BATT: F1.1, J1.1 (Pin_1)
- new net BATT_Level: R1.2, R2.2
- new net GND: J1.2 (Pin_2), R2.1, U2.2 (-VIN), U2.5 (-VOUT), U3.2 (-VIN), U3.5 (-VOUT), U4.2 (-VIN), U4.5 (-VOUT)
- new net PWR_MOTOR: R1.1, SW1.2, U2.1 (+VIN), U3.1 (+VIN), U4.1 (+VIN)
- no-connect marks 0 -> 3
Other:
- note added: "Voltage Divider"
- note added: "Voltage supply"
- company: (none) -> Ginobeano
- title: (none) -> BeanBike Controller Power

Commit message: PCB v1
Whole lotta stuff
Parts:
- removed SW1: SW_Push, symbol Switch:SW_Push
- removed U2: JTD2048S3V3, Converter_DCDC:Converter_DCDC_XP_POWER_JTDxxxxxxx_THT, symbol Converter_DCDC:JTD2048S3V3
- removed U3: JTD2048S05, Converter_DCDC:Converter_DCDC_XP_POWER_JTDxxxxxxx_THT, symbol Converter_DCDC:JTD2048S05
- removed U4: JTD2048S12, Converter_DCDC:Converter_DCDC_XP_POWER_JTDxxxxxxx_THT, symbol Converter_DCDC:JTD2048S12
- F1: footprint (none) -> Fuse:Fuse_1206_3216Metric
- J1: footprint (none) -> Connector_Wire:SolderWire-2sqmm_1x02_P7.8mm_D2mm_OD3.9mm
- R1: renamed from R2; footprint (none) -> Resistor_SMD:R_0603_1608Metric
- R2: renamed from R1; footprint (none) -> Resistor_SMD:R_0603_1608Metric
Connections:
- net PWR_MOTOR: now also F1.2
- no-connect marks 3 -> 0
Other:
- added sheet 12v (beanbike_controller_12v.kicad_sch)
- added sheet 24v (beanbike_controller_24v.kicad_sch)
- added sheet 3.3v (beanbike_controller_3.3v.kicad_sch)
- added sheet 5v (beanbike_controller_5v.kicad_sch)
- moved on the sheet: F1, J1, R1, R2

Commit message: PCB v2
Other:
- removed sheet 12v
- removed sheet 24v
- sheet 5v ports: added BATT; removed 12v
