File: KiCad/BeanBike/Controller/beanbike_controller_3.3v.kicad_sch (KiCad schematic)
At the start: 11 parts

Commit message: PCB v2
Parts:
- renumbered C23 to C13, C24 to C14, C25 to C15, C26 to C16, C27 to C17, L4 to L2, PS4 to PS2, R29 to R21, R30 to R22, R31 to R23, R32 to R24
Connections:
- net 5v: now also C14.1
- net GND: now also C13.2
Other:
- moved on the sheet: C13, C14
Changed lines of the file:
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@@
+	)
+	(junction
+		(at 88.9 93.98)
+		(diameter 0)
+		(color 0 0 0 0)
 	)
 	(junction
@@
 	)
 	(junction
+		(at 88.9 109.22)
+		(diameter 0)
+		(color 0 0 0 0)
+	)
+	(junction
 		(at 191.77 124.46)
 		(diameter 0)
@@
 	(wire
 		(pts
+			(xy 81.28 97.79) (xy 81.28 93.98)
+		)
+		(stroke
+			(width 0)
+			(type default)
+		)
+	)
+	(wire
+		(pts
 			(xy 171.45 124.46) (xy 142.24 124.46)
 		)
@@
 	(wire
 		(pts
-			(xy 81.28 109.22) (xy 95.25 109.22)
-		)
-		(stroke
-			(width 0)
-			(type default)
-		)
-	)
-	(wire
-		(pts
 			(xy 105.41 93.98) (xy 105.41 100.33)
 		)
@@
 	(wire
 		(pts
+			(xy 81.28 105.41) (xy 81.28 109.22)
+		)
+		(stroke
+			(width 0)
+			(type default)
+		)
+	)
+	(wire
+		(pts
 			(xy 105.41 107.95) (xy 105.41 105.41)
 		)
@@
 	(wire
 		(pts
+			(xy 88.9 105.41) (xy 88.9 109.22)
+		)
+		(stroke
+			(width 0)
+			(type default)
+		)
+	)
+	(wire
+		(pts
 			(xy 168.91 95.25) (xy 168.91 97.79)
 		)
@@
 	(wire
 		(pts
-			(xy 81.28 93.98) (xy 95.25 93.98)
+			(xy 81.28 109.22) (xy 88.9 109.22)
+		)
+		(stroke
+			(width 0)
+			(type default)
+		)
+	)
+	(wire
+		(pts
+			(xy 88.9 93.98) (xy 95.25 93.98)
+		)
+		(stroke
+			(width 0)
+			(type default)
+		)
+	)
+	(wire
+		(pts
+			(xy 81.28 93.98) (xy 88.9 93.98)
 		)
 		(stroke
@@
 	(wire
 		(pts
+			(xy 88.9 109.22) (xy 95.25 109.22)
+		)
+		(stroke
+			(width 0)
+			(type default)
+		)
+	)
+	(wire
+		(pts
 			(xy 114.3 97.79) (xy 114.3 124.46)
 		)
@@
 		(pts
 			(xy 177.8 95.25) (xy 172.72 95.25)
+		)
+		(stroke
+			(width 0)
+			(type default)
+		)
+	)
+	(wire
+		(pts
+			(xy 88.9 93.98) (xy 88.9 97.79)
 		)
 		(stroke
@@
 		(dnp no)
 		(fields_autoplaced yes)
-		(property "Reference" "R30"
+		(property "Reference" "R22"
 			(at 187.96 96.52 90)
 			(effects
@@
 			(project "Controller"
 				(path "/645e8d68-d9e1-48b3-98a5-3b81aa58d1ea/ceef88aa-c829-4630-8455-6c437ac60286/50bbad7b-d737-4b31-afb1-bf79d85d411a"
-					(reference "R30")
-					(unit 1)
-				)
-				(path "/645e8d68-d9e1-48b3-98a5-3b81aa58d1ea/ceef88aa-c829-4630-8455-6c437ac60286/a3eae8f7-1220-4fa3-bfaf-a2df91ade4b0"
-					(reference "R16")
+					(reference "R22")
 					(unit 1)
 				)
@@
 		(dnp no)
 		(fields_autoplaced yes)
-		(property "Reference" "PS4"
+		(property "Reference" "PS2"
 			(at 142.24 87.63 0)
 			(effects
@@
 			(project "Controller"
 				(path "/645e8d68-d9e1-48b3-98a5-3b81aa58d1ea/ceef88aa-c829-4630-8455-6c437ac60286/50bbad7b-d737-4b31-afb1-bf79d85d411a"
-					(reference "PS4")
-					(unit 1)
-				)
-				(path "/645e8d68-d9e1-48b3-98a5-3b81aa58d1ea/ceef88aa-c829-4630-8455-6c437ac60286/a3eae8f7-1220-4fa3-bfaf-a2df91ade4b0"
-					(reference "PS1")
+					(reference "PS2")
 					(unit 1)
 				)
@@
 		(dnp no)
 		(fields_autoplaced yes)
-		(property "Reference" "L4"
+		(property "Reference" "L2"
 			(at 181.61 90.17 90)
 			(effects
@@
 			(project "Controller"
 				(path "/645e8d68-d9e1-48b3-98a5-3b81aa58d1ea/ceef88aa-c829-4630-8455-6c437ac60286/50bbad7b-d737-4b31-afb1-bf79d85d411a"
-					(reference "L4")
-					(unit 1)
-				)
-				(path "/645e8d68-d9e1-48b3-98a5-3b81aa58d1ea/ceef88aa-c829-4630-8455-6c437ac60286/a3eae8f7-1220-4fa3-bfaf-a2df91ade4b0"
-					(reference "L1")
+					(reference "L2")
 					(unit 1)
 				)
@@
 		(dnp no)
 		(fields_autoplaced yes)
-		(property "Reference" "#PWR035"
+		(property "Reference" "#PWR028"
 			(at 71.12 130.81 0)
 			(effects
@@
 			(project "Controller"
 				(path "/645e8d68-d9e1-48b3-98a5-3b81aa58d1ea/ceef88aa-c829-4630-8455-6c437ac60286/50bbad7b-d737-4b31-afb1-bf79d85d411a"
-					(reference "#PWR035")
-					(unit 1)
-				)
-				(path "/645e8d68-d9e1-48b3-98a5-3b81aa58d1ea/ceef88aa-c829-4630-8455-6c437ac60286/a3eae8f7-1220-4fa3-bfaf-a2df91ade4b0"
-					(reference "#PWR06")
+					(reference "#PWR028")
 					(unit 1)
 				)
@@
 		(on_board yes)
 		(dnp no)
-		(property "Reference" "C27"
+		(property "Reference" "C17"
 			(at 229.87 109.22 90)
 			(effects
@@
 			(project "Controller"
 				(path "/645e8d68-d9e1-48b3-98a5-3b81aa58d1ea/ceef88aa-c829-4630-8455-6c437ac60286/50bbad7b-d737-4b31-afb1-bf79d85d411a"
-					(reference "C27")
-					(unit 1)
-				)
-				(path "/645e8d68-d9e1-48b3-98a5-3b81aa58d1ea/ceef88aa-c829-4630-8455-6c437ac60286/a3eae8f7-1220-4fa3-bfaf-a2df91ade4b0"
-					(reference "C20")
+					(reference "C17")
 					(unit 1)
 				)
@@
 		(dnp no)
 		(fields_autoplaced yes)
-		(property "Reference" "#PWR036"
+		(property "Reference" "#PWR029"
 			(at 247.65 102.87 0)
 			(effects
@@
 			(project ""
 				(path "/645e8d68-d9e1-48b3-98a5-3b81aa58d1ea/ceef88aa-c829-4630-8455-6c437ac60286/50bbad7b-d737-4b31-afb1-bf79d85d411a"
-					(reference "#PWR036")
+					(reference "#PWR029")
 					(unit 1)
 				)
@@
 		(dnp no)
 		(fields_autoplaced yes)
-		(property "Reference" "R29"
+		(property "Reference" "R21"
 			(at 173.99 111.7599 0)
 			(effects
@@
 			(project "Controller"
 				(path "/645e8d68-d9e1-48b3-98a5-3b81aa58d1ea/ceef88aa-c829-4630-8455-6c437ac60286/50bbad7b-d737-4b31-afb1-bf79d85d411a"
-					(reference "R29")
-					(unit 1)
-				)
-				(path "/645e8d68-d9e1-48b3-98a5-3b81aa58d1ea/ceef88aa-c829-4630-8455-6c437ac60286/a3eae8f7-1220-4fa3-bfaf-a2df91ade4b0"
-					(reference "R14")
+					(reference "R21")
 					(unit 1)
 				)
@@
 		(dnp no)
 		(fields_autoplaced yes)
-		(property "Reference" "C25"
+		(property "Reference" "C15"
 			(at 99.06 100.3299 0)
 			(effects
@@
 			(project "Controller"
 				(path "/645e8d68-d9e1-48b3-98a5-3b81aa58d1ea/ceef88aa-c829-4630-8455-6c437ac60286/50bbad7b-d737-4b31-afb1-bf79d85d411a"
-					(reference "C25")
-					(unit 1)
-				)
-				(path "/645e8d68-d9e1-48b3-98a5-3b81aa58d1ea/ceef88aa-c829-4630-8455-6c437ac60286/a3eae8f7-1220-4fa3-bfaf-a2df91ade4b0"
-					(reference "C18")
+					(reference "C15")
 					(unit 1)
 				)
@@
 	(symbol
 		(lib_id "Device:C")
-		(at 81.28 97.79 0)
+		(at 81.28 101.6 0)
 		(unit 1)
 		(exclude_from_sim no)
@@
 		(dnp no)
 		(fields_autoplaced yes)
-		(property "Reference" "C23"
-			(at 85.09 96.5199 0)
+		(property "Reference" "C13"
+			(at 85.09 100.3299 0)
 			(effects
 				(font
@@
 		)
 		(property "Value" "2.2uF"
-			(at 85.09 99.0599 0)
+			(at 85.09 102.8699 0)
 			(effects
 				(font
@@
 		)
 		(property "Footprint" "Capacitor_SMD:C_0201_0603Metric"
-			(at 82.2452 101.6 0)
+			(at 82.2452 105.41 0)
 			(effects
 				(font
@@
 		)
 		(property "Datasheet" "~"
-			(at 81.28 97.79 0)
+			(at 81.28 101.6 0)
 			(effects
 				(font
@@
 		)
 		(property "Description" "Unpolarized capacitor"
-			(at 81.28 97.79 0)
+			(at 81.28 101.6 0)
 			(effects
 				(font
@@
 			(project "Controller"
 				(path "/645e8d68-d9e1-48b3-98a5-3b81aa58d1ea/ceef88aa-c829-4630-8455-6c437ac60286/50bbad7b-d737-4b31-afb1-bf79d85d411a"
-					(reference "C23")
-					(unit 1)
-				)
-				(path "/645e8d68-d9e1-48b3-98a5-3b81aa58d1ea/ceef88aa-c829-4630-8455-6c437ac60286/a3eae8f7-1220-4fa3-bfaf-a2df91ade4b0"
-					(reference "C7")
+					(reference "C13")
 					(unit 1)
 				)
@@
 		(dnp no)
 		(fields_autoplaced yes)
-		(property "Reference" "R32"
+		(property "Reference" "R24"
 			(at 218.44 109.2199 0)
 			(effects
@@
 			(project "Controller"
 				(path "/645e8d68-d9e1-48b3-98a5-3b81aa58d1ea/ceef88aa-c829-4630-8455-6c437ac60286/50bbad7b-d737-4b31-afb1-bf79d85d411a"
-					(reference "R32")
-					(unit 1)
-				)
-				(path "/645e8d68-d9e1-48b3-98a5-3b81aa58d1ea/ceef88aa-c829-4630-8455-6c437ac60286/a3eae8f7-1220-4fa3-bfaf-a2df91ade4b0"
-					(reference "R26")
+					(reference "R24")
 					(unit 1)
 				)
@@
 		(on_board yes)
 		(dnp no)
-		(property "Reference" "C26"
+		(property "Reference" "C16"
 			(at 168.91 92.71 90)
 			(effects
@@
 			(project "Controller"
 				(path "/645e8d68-d9e1-48b3-98a5-3b81aa58d1ea/ceef88aa-c829-4630-8455-6c437ac60286/50bbad7b-d737-4b31-afb1-bf79d85d411a"
-					(reference "C26")
-					(unit 1)
-				)
-				(path "/645e8d68-d9e1-48b3-98a5-3b81aa58d1ea/ceef88aa-c829-4630-8455-6c437ac60286/a3eae8f7-1220-4fa3-bfaf-a2df91ade4b0"
-					(reference "C19")
+					(reference "C16")
 					(unit 1)
 				)
@@
 	(symbol
 		(lib_id "Device:C")
-		(at 81.28 105.41 0)
+		(at 88.9 101.6 0)
 		(unit 1)
 		(exclude_from_sim no)
@@
 		(dnp no)
 		(fields_autoplaced yes)
-		(property "Reference" "C24"
-			(at 85.09 104.1399 0)
+		(property "Reference" "C14"
+			(at 92.71 100.3299 0)
 			(effects
 				(font
@@
 		)
 		(property "Value" "2.2uF"
-			(at 85.09 106.6799 0)
+			(at 92.71 102.8699 0)
 			(effects
 				(font
@@
 		)
 		(property "Footprint" "Capacitor_SMD:C_0201_0603Metric"
-			(at 82.2452 109.22 0)
+			(at 89.8652 105.41 0)
 			(effects
 				(font
@@
 		)
 		(property "Datasheet" "~"
-			(at 81.28 105.41 0)
+			(at 88.9 101.6 0)
 			(effects
 				(font
@@
 		)
 		(property "Description" "Unpolarized capacitor"
-			(at 81.28 105.41 0)
+			(at 88.9 101.6 0)
 			(effects
 				(font
@@
 			(project "Controller"
 				(path "/645e8d68-d9e1-48b3-98a5-3b81aa58d1ea/ceef88aa-c829-4630-8455-6c437ac60286/50bbad7b-d737-4b31-afb1-bf79d85d411a"
-					(reference "C24")
-					(unit 1)
-				)
-				(path "/645e8d68-d9e1-48b3-98a5-3b81aa58d1ea/ceef88aa-c829-4630-8455-6c437ac60286/a3eae8f7-1220-4fa3-bfaf-a2df91ade4b0"
-					(reference "C10")
+					(reference "C14")
 					(unit 1)
 				)
@@
 		(dnp no)
 		(fields_autoplaced yes)
-		(property "Reference" "R31"
+		(property "Reference" "R23"
 			(at 218.44 97.7899 0)
 			(effects
@@
 			(project "Controller"
 				(path "/645e8d68-d9e1-48b3-98a5-3b81aa58d1ea/ceef88aa-c829-4630-8455-6c437ac60286/50bbad7b-d737-4b31-afb1-bf79d85d411a"
-					(reference "R31")
+					(reference "R23")
 					(unit 1)
 				)
-				(path "/645e8d68-d9e1-48b3-98a5-3b81aa58d1ea/ceef88aa-c829-4630-8455-6c437ac60286/a3eae8f7-1220-4fa3-bfaf-a2df91ade4b0"
-					(reference "R25")
-					(unit 1)
-				)

Commit message: PCBv2 Finish
Other:
- moved on the sheet: C17
Changed lines of the file:
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@@
+	)
+	(junction
+		(at 226.06 95.25)
+		(diameter 0)
+		(color 0 0 0 0)
 	)
 	(junction
@@
 	)
 	(junction
-		(at 237.49 102.87)
-		(diameter 0)
-		(color 0 0 0 0)
-	)
-	(junction
 		(at 171.45 124.46)
 		(diameter 0)
@@
 	(wire
 		(pts
+			(xy 226.06 95.25) (xy 215.9 95.25)
+		)
+		(stroke
+			(width 0)
+			(type default)
+		)
+	)
+	(wire
+		(pts
 			(xy 171.45 116.84) (xy 171.45 124.46)
 		)
@@
 	(wire
 		(pts
+			(xy 226.06 95.25) (xy 226.06 102.87)
+		)
+		(stroke
+			(width 0)
+			(type default)
+		)
+	)
+	(wire
+		(pts
 			(xy 168.91 95.25) (xy 168.91 97.79)
 		)
@@
 	(wire
 		(pts
-			(xy 237.49 95.25) (xy 215.9 95.25)
+			(xy 237.49 95.25) (xy 226.06 95.25)
 		)
 		(stroke
@@
 	(wire
 		(pts
-			(xy 237.49 113.03) (xy 237.49 124.46)
-		)
-		(stroke
-			(width 0)
-			(type default)
-		)
-	)
-	(wire
-		(pts
 			(xy 124.46 95.25) (xy 114.3 95.25)
 		)
@@
 	(wire
 		(pts
-			(xy 237.49 124.46) (xy 215.9 124.46)
+			(xy 226.06 124.46) (xy 215.9 124.46)
 		)
 		(stroke
@@
 	(wire
 		(pts
-			(xy 237.49 102.87) (xy 237.49 105.41)
-		)
-		(stroke
-			(width 0)
-			(type default)
-		)
-	)
-	(wire
-		(pts
 			(xy 124.46 107.95) (xy 105.41 107.95)
 		)
@@
 		(pts
 			(xy 191.77 124.46) (xy 171.45 124.46)
+		)
+		(stroke
+			(width 0)
+			(type default)
+		)
+	)
+	(wire
+		(pts
+			(xy 226.06 110.49) (xy 226.06 124.46)
 		)
 		(stroke
@@
 	(symbol
 		(lib_id "Device:C")
-		(at 237.49 109.22 180)
+		(at 226.06 106.68 180)
 		(unit 1)
 		(exclude_from_sim no)
@@
 		(dnp no)
 		(property "Reference" "C17"
-			(at 229.87 109.22 90)
+			(at 218.44 106.68 90)
 			(effects
 				(font
@@
 		)
 		(property "Value" "22uF"
-			(at 241.3 109.22 90)
+			(at 229.87 106.68 90)
 			(effects
 				(font
@@
 		)
 		(property "Footprint" "Capacitor_SMD:C_0603_1608Metric"
-			(at 236.5248 105.41 0)
+			(at 225.0948 102.87 0)
 			(effects
 				(font
@@
 		)
 		(property "Datasheet" "~"
-			(at 237.49 109.22 0)
+			(at 226.06 106.68 0)
 			(effects
 				(font
@@
 		)
 		(property "Description" "Unpolarized capacitor"
-			(at 237.49 109.22 0)
-			(effects
-				(font
+			(at 226.06 106.68 0)
+			(effects
+				(font
