File: KiCad/BeanBike/Controller/beanbike_controller_5v.kicad_sch (KiCad schematic)
At the start: 11 parts

Commit message: PCB v2
Parts:
- added C12: 22uF, Capacitor_SMD:C_0603_1608Metric, symbol Device:C
- L1: renamed from L3; value L -> 8.2uH 68mOhm; footprint 0630CDMCCDS_3R3MC:IND_CCDS-3R3MC_SUM -> 74438357082:WE-MAPI_4030
- R17: renamed from R25; value 21.5k -> 46.4k
- renumbered C21 to C10, C22 to C11, C18 to C7, C19 to C8, C20 to C9, PS3 to PS1, R26 to R18, R27 to R19, R28 to R20
Connections:
- net 12v is gone; now on net BATT: C7.1, C9.1, PS1.3 (EN), PS1.5 (VIN_1), PS1.6 (VIN_2)
- net GND is gone; now on net +5V: C11.1, C8.2, C9.2, PS1.1 (GND_1), PS1.13 (EP), PS1.2 (GND_2), R17.2, R18.2, R20.1
- net +5V: now also C7.2, C12.1, C12.2
- net BATT: now reaches C8.1
- net BATT: no longer C7.2
Other:
- moved on the sheet: C11, C7, C8

Commit message: PCBv2 Finish
Connections:
- net +5V: no longer C11.1, C12.1, C7.2, C8.2, C9.2, PS1.1 (GND_1), PS1.13 (EP), PS1.2 (GND_2), R17.2, R18.2, R20.1
- new net GND: C11.1, C12.1, C7.2, C8.2, C9.2, PS1.1 (GND_1), PS1.13 (EP), PS1.2 (GND_2), R17.2, R18.2, R20.1
Changed lines of the file:
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@@
-	)
-	(junction
-		(at 231.14 124.46)
-		(diameter 0)
-		(color 0 0 0 0)
 	)
 	(junction
@@
 	)
 	(junction
-		(at 237.49 102.87)
-		(diameter 0)
-		(color 0 0 0 0)
-	)
-	(junction
 		(at 223.52 95.25)
 		(diameter 0)
@@
 	(wire
 		(pts
-			(xy 237.49 102.87) (xy 237.49 124.46)
-		)
-		(stroke
-			(width 0)
-			(type default)
-		)
-	)
-	(wire
-		(pts
 			(xy 124.46 95.25) (xy 114.3 95.25)
 		)
@@
 		)
 		(stroke
-			(width 0)
-			(type default)
-		)
-	)
-	(wire
-		(pts
-			(xy 237.49 124.46) (xy 231.14 124.46)
-		)
-		(stroke
