File: KiCad/BeanBike/Controller/Controller.kicad_pcb (KiCad board)
At the start: 4 copper layers, 61.1 x 61.2 mm, 86 parts, among them J1 XT80 Male, J2 Motor Conn, J3 Throttle Conn, J4 PAS Conn, J5 Display Conn, J6 Brake Conn, Q1 PHASE A HIGH, Q2 PHASE B HIGH, Q3 PHASE C HIGH, Q4 PHASE A LOW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

Commit message: PCB v2
Parts:
- removed C18, C19, C23, C24: 2.2uF, Capacitor_SMD:C_0201_0603Metric
- removed C20, C25: 100nF, Capacitor_SMD:C_0201_0603Metric
- removed C21, C26: 100nf, Capacitor_SMD:C_0201_0603Metric
- removed C22, C27: 22uF, Capacitor_SMD:C_0603_1608Metric
- removed L3: L, 0630CDMCCDS_3R3MC:IND_CCDS-3R3MC_SUM
- removed L4: L, PA4332_152NLT:IND_PA4332.152NLT
- removed PS3, PS4: LMR38025SQDRRRQ1, LMR380:SON50P300X300X80-13N
- removed R25, R29: 21.5k, Resistor_SMD:R_0402_1005Metric
- removed R26, R28, R30, R32: 10k, Resistor_SMD:R_0603_1608Metric
- removed R27: 40.2k, Resistor_SMD:R_0402_1005Metric
- removed R31: 23.2k, Resistor_SMD:R_0805_2012Metric
- C11, C12: value 4.7uF -> 22uF; footprint Capacitor_SMD:C_0201_0603Metric -> Capacitor_SMD:C_0603_1608Metric
- C17: value 10uF -> 22uF; footprint Capacitor_SMD:C_0402_1005Metric -> Capacitor_SMD:C_0603_1608Metric
- L1: value L -> 8.2uH 68mOhm; footprint Inductor_SMD:L_12x12mm_H8mm -> 74438357082:WE-MAPI_4030
- L2: footprint IHLP4040DZER5R6M01:IND_IHLP-4040DZ_VIS -> PA4332_152NLT:IND_PA4332.152NLT
- R17: value 21.5k -> 46.4k
- R19: value 232k -> 40.2k
- R23: value 110k -> 23.2k; footprint Resistor_SMD:R_0402_1005Metric -> Resistor_SMD:R_0805_2012Metric
- moved R16 58.0 mm to (149.2, 89.5)
- moved R15 57.7 mm to (149.1, 87.9)
- moved D1 55.1 mm to (152.5, 84.0), turned to -90 degrees
- moved R11 54.8 mm to (149.3, 82.2)
- moved R12 54.6 mm to (149.2, 83.8)
- moved R13 54.6 mm to (149.2, 85.0)
- moved R14 54.5 mm to (149.2, 86.5)
- moved R10 54.1 mm to (146.0, 89.5)
- moved R5 53.9 mm to (146.0, 82.0)
- moved R6 53.9 mm to (146.0, 83.5)
- moved R7 53.9 mm to (146.0, 85.0)
- moved R8 53.9 mm to (146.0, 86.5)
- moved R9 53.9 mm to (146.0, 88.0)
- moved U4 53.3 mm to (139.9, 84.5)
- moved D2 52.4 mm to (152.5, 80.6), turned to 90 degrees
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Connections:
- C11 pad 1: +24V -> DISPLAY_5V
- C11 pad 2: Net-(C11-Pad2) -> DISPLAY_5V
- C12 pad 1: BRAKE_GND -> DISPLAY_5V
- C12 pad 2: +24V -> DISPLAY_5V
- C13 pad 1: +24V -> DISPLAY_5V
- C13 pad 2: Net-(C13-Pad2) -> BRAKE_GND
- C14 pad 1: Net-(C13-Pad2) -> DISPLAY_5V
- C15 pad 1: +24V -> DISPLAY_5V
- C17 pad 2: +12V -> +3.3V
- C7 pad 2: Net-(C7-Pad2) -> DISPLAY_5V
- C8 pad 1: Net-(C7-Pad2) -> PWR_MOTOR
- C8 pad 2: BRAKE_GND -> DISPLAY_5V
- C9 pad 2: BRAKE_GND -> DISPLAY_5V
- L1 pad 2: Net-(C11-Pad2) -> DISPLAY_5V
- L2 pad 2: +12V -> +3.3V
- PS1 pad 1: BRAKE_GND -> DISPLAY_5V
- PS1 pad 13: BRAKE_GND -> DISPLAY_5V
- PS1 pad 2: BRAKE_GND -> DISPLAY_5V
- PS2 pad 3: +24V -> DISPLAY_5V
- PS2 pad 5: +24V -> DISPLAY_5V
- PS2 pad 6: +24V -> DISPLAY_5V
- R17 pad 2: BRAKE_GND -> DISPLAY_5V
- R18 pad 2: BRAKE_GND -> DISPLAY_5V
- R19 pad 2: Net-(C11-Pad2) -> DISPLAY_5V
- R20 pad 1: BRAKE_GND -> DISPLAY_5V
- R23 pad 2: +12V -> +3.3V
Routing:
- net +3.3V: track 131.1 -> 0.00 mm, vias 2 -> 0
- net DISPLAY_5V: track 123.0 -> 0.00 mm, vias 4 -> 0
- net PWR_MOTOR: track 114.7 -> 0.00 mm
- net MOTOR_HALL_5V: track 112.2 -> 3.00 mm, vias 5 -> 0
- net MCU-GPIO4: track 95.9 -> 0.00 mm, vias 5 -> 0
- net MCU-TX: track 66.1 -> 0.00 mm, vias 3 -> 0
- net BRAKE_SIGNAL: track 61.9 -> 0.00 mm, vias 3 -> 0
- net MOTOR_PHASE_C: track 60.5 -> 0.00 mm, vias 1 -> 0
- net MCU-GPIO21: track 60.5 -> 0.00 mm, vias 4 -> 0
- net MCU-GPIO22: track 59.4 -> 0.00 mm, vias 3 -> 0
- net BATT_Level: track 59.0 -> 0.00 mm, vias 2 -> 0
- net MCU-RX: track 58.2 -> 0.00 mm, vias 4 -> 0
- net MCU-Boot: track 51.7 -> 0.00 mm, vias 3 -> 0
- net /Motor/Control/FAULT: track 54.6 -> 5.76 mm, vias 4 -> 0
- net MOTOR_PHASE_B: track 46.5 -> 0.00 mm, vias 1 -> 0
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- added copper zone on In4.Cu, net PWR_MOTOR
- removed copper zone on F.Cu, net BRAKE_GND
Other:
- board size 61.1 x 61.2 mm -> 49.8 x 70.4 mm
- copper layers 4 -> 6
- board text removed: "BEAN BIKE"
- board text removed: "BeanBike Controller 48v 1200w"
- board text removed: "By: Ginobeano"
- board text removed: "Make sure to install heatsinks!!!"

Commit message: PCBv2 Finish
Parts:
- removed C1: 0.1uF 35v, Capacitor_SMD:C_0201_0603Metric
- removed C2: 1uF 6.3V cermaic, Capacitor_SMD:C_0402_1005Metric
- removed C3, C4: 0.1uF ceramic, Capacitor_SMD:C_0201_0603Metric
- removed C5: 1uf, Capacitor_SMD:C_0402_1005Metric
- removed C6: WCAP-ASLI_4X5.5, 865080340001:WCAP-ASLI_4X5.5_DXL_
- removed D1, D2: D, Diode_SMD:D_SOD-323
- removed R10, R6, R7, R8, R9: 10k, Resistor_SMD:R_0603_1608Metric
- removed R11, R12, R13, R14, R15, R16: 1k, Resistor_SMD:R_0402_1005Metric
- removed U2: DRV8308, Package_DFN_QFN:Texas_RHA0040E_VQFN-40-1EP_6x6mm_P0.5mm_EP3.52x2.62mm
- removed U3, U4: TXB0108DQSR, Package_SON:USON-20_2x4mm_P0.4mm
- added C18: 0.1uF, Capacitor_SMD:C_0201_0603Metric, F.Cu at (137.6, 106.6)
- added C19: >10uF, Capacitor_SMD:C_0603_1608Metric, F.Cu at (135.8, 107.0)
- added C20: 1uF, Capacitor_SMD:C_0201_0603Metric, F.Cu at (135.5, 104.8)
- added C21: 47nF, Capacitor_SMD:C_0201_0603Metric, F.Cu at (134.6, 107.1)
- added C22: 1uF, Capacitor_SMD:C_0201_0603Metric, F.Cu at (128.9, 109.7)
- added C23: 1uF, Capacitor_SMD:C_0201_0603Metric, F.Cu at (129.9, 109.0)
- added C24: 0.1uF, Capacitor_SMD:C_0201_0603Metric, F.Cu at (120.9, 104.4)
- added R25: 73k, Resistor_SMD:R_0603_1608Metric, F.Cu at (120.1, 108.5)
- added R26: 73k, Resistor_SMD:R_0603_1608Metric, F.Cu at (120.9, 106.2)
- added U5: DRV8353SRTAT, MOTORIC:RTA0040B, F.Cu at (127.3, 105.1)
- R3: value WSLP39212L500FEA -> CSS2H-2512R-1L00F; footprint WSLP39212L500FEA:RES_WSLP39212L500FEA -> Resistor_SMD:R_2512_6332Metric
- R4, R5: value 10k -> CSS2H-2512R-1L00F; footprint Resistor_SMD:R_0603_1608Metric -> Resistor_SMD:R_2512_6332Metric
- moved R4 26.8 mm to (143.8, 105.2)
- moved Q6 21.5 mm to (119.9, 95.4), turned to 180 degrees
- moved Q5 21.5 mm to (130.4, 95.4), turned to 180 degrees
- moved Q4 21.4 mm to (141.1, 95.5), turned to 180 degrees
- moved R3 19.4 mm to (143.8, 109.0), turned to 0 degrees
- moved R5 19.3 mm to (143.8, 101.2), turned to 0 degrees
- moved Q1 19.1 mm to (136.1, 115.0), turned to 0 degrees
- moved Q3 19.1 mm to (114.8, 114.9), turned to 0 degrees
- moved Q2 19.1 mm to (125.4, 114.9), turned to 0 degrees
- moved R21 0.35 mm to (125.7, 134.1)
- moved R18 0.20 mm to (116.8, 125.4)
Connections:
- C11 pad 1: DISPLAY_5V -> BRAKE_GND
- C12 pad 1: DISPLAY_5V -> BRAKE_GND
- C7 pad 2: DISPLAY_5V -> BRAKE_GND
- C8 pad 2: DISPLAY_5V -> BRAKE_GND
- C9 pad 2: DISPLAY_5V -> BRAKE_GND
- J3 pad 3: MCU-GPIO21 -> MCU-GPIO34
- J4 pad 3: MCU-GPIO22 -> MCU-GPIO35
- J5 pad 5: MCU-GPIO4 -> MCU-Reset
- PS1 pad 1: DISPLAY_5V -> BRAKE_GND
- PS1 pad 13: DISPLAY_5V -> BRAKE_GND
- PS1 pad 2: DISPLAY_5V -> BRAKE_GND
- Q1 pad 2: MOTOR_PHASE_A -> PWR_MOTOR
- Q1 pad 3: PWR_MOTOR -> MOTOR_PHASE_A
- Q2 pad 2: MOTOR_PHASE_B -> PWR_MOTOR
- Q2 pad 3: PWR_MOTOR -> MOTOR_PHASE_B
- Q3 pad 2: MOTOR_PHASE_C -> PWR_MOTOR
- Q3 pad 3: PWR_MOTOR -> MOTOR_PHASE_C
- Q4 pad 2: MOTOR_PHASE_A -> BRAKE_GND
- Q4 pad 3: BRAKE_GND -> MOTOR_PHASE_A
- Q5 pad 2: MOTOR_PHASE_B -> BRAKE_GND
- Q5 pad 3: BRAKE_GND -> MOTOR_PHASE_B
- Q6 pad 2: MOTOR_PHASE_C -> BRAKE_GND
- Q6 pad 3: BRAKE_GND -> MOTOR_PHASE_C
- R17 pad 2: DISPLAY_5V -> BRAKE_GND
- R18 pad 2: DISPLAY_5V -> BRAKE_GND
- R20 pad 1: DISPLAY_5V -> BRAKE_GND
- R3 pad 1: BRAKE_GND -> MOTOR_PHASE_C
- R4 pad 1: +3.3V -> MOTOR_PHASE_B
- R4 pad 2: MCU-GPIO20 -> BRAKE_GND
- R5 pad 1: MOTOR_HALL_5V -> MOTOR_PHASE_A
- R5 pad 2: Net-(U4-B1) -> BRAKE_GND
- U1 pad 27: MCU-GPIO16 -> BATT_Level
- U1 pad 3: MCU-GPIO4 -> MCU-Reset
- U1 pad 37: BRAKE_SIGNAL -> MCU-GPIO23
- U1 pad 8: BATT_Level -> BRAKE_SIGNAL
Routing:
- net +3.3V: track 0.00 -> 77.4 mm
- net BATT_Level: track 0.00 -> 67.5 mm, vias 0 -> 2
- net DISPLAY_5V: track 0.00 -> 64.5 mm
- net MCU-GPIO18: track 0.00 -> 53.1 mm, vias 0 -> 2
- net MCU-GPIO19: track 0.00 -> 52.0 mm, vias 0 -> 2
- net MCU-GPIO33: track 0.00 -> 46.8 mm, vias 0 -> 2
- net MCU-GPIO23: track 0.00 -> 42.1 mm, vias 0 -> 2
- net MCU-GPIO25: track 0.00 -> 40.8 mm, vias 0 -> 2
- net MCU-Boot: track 0.00 -> 40.0 mm
- net MCU-GPIO22: track 0.00 -> 38.7 mm, vias 0 -> 2
- net BRAKE_SIGNAL: track 0.00 -> 36.5 mm, vias 0 -> 1
- net MCU-GPIO26: track 0.00 -> 34.3 mm, vias 0 -> 2
- net MCU-GPIO17: track 0.00 -> 33.1 mm, vias 0 -> 3
- net MCU-GPIO5: track 0.00 -> 32.5 mm, vias 0 -> 2
- net MCU-GPIO14: track 0.00 -> 32.1 mm, vias 0 -> 2
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- added copper zone on In3.Cu, net MOTOR_PHASE_A
- added copper zone on In2.Cu, net MOTOR_PHASE_B
- added copper zone on In1.Cu, net MOTOR_PHASE_C

Commit message: Silkscreen
Other:
- board text added: "Bean Bike"
- board text added: "BeanBike Controller 48v 1200w"
- board text added: "GINOBEANO"
Changed lines of the file:
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@@
 		(layer "Edge.Cuts")
+	)
+	(gr_text "GINOBEANO\n"
+		(at 140.05 86.95 0)
+		(layer "F.SilkS")
+		(effects
+			(font
+				(size 1 1)
+				(thickness 0.1)
+			)
+			(justify left bottom)
+		)
+	)
+	(gr_text "BeanBike\nController\n48v 1200w"
+		(at 140.15 76.55 0)
+		(layer "F.SilkS")
+		(effects
+			(font
+				(size 1 1)
+				(thickness 0.1)
+			)
+			(justify left bottom)
+		)
+	)
+	(gr_text "Bean\nBike\n"
+		(at 157.3 127.1 0)
+		(layer "B.SilkS")
+		(effects
+			(font
+				(size 15 15)
+				(thickness 1.875)
+			)
+			(justify left bottom mirror)
+		)
 	)
 	(segment

Commit message: More Firmware
😄
Parts:
- added R10: 10k, Resistor_SMD:R_0603_1608Metric, F.Cu at (149.7, 86.8)
- added R11: 18k, Resistor_SMD:R_0603_1608Metric, F.Cu at (149.7, 85.3)
- added R6: 10k, Resistor_SMD:R_0603_1608Metric, F.Cu at (149.7, 92.8)
- added R7: 18k, Resistor_SMD:R_0603_1608Metric, F.Cu at (149.7, 91.2)
- added R8: 10k, Resistor_SMD:R_0603_1608Metric, F.Cu at (149.7, 89.8)
- added R9: 18k, Resistor_SMD:R_0603_1608Metric, F.Cu at (149.7, 88.3)
- moved J2 0.85 mm to (150.9, 97.9)
Connections:
- J2 pad 4: MOTOR_HALL_5V -> DISPLAY_5V
- R26 pad 2: Net-(U5-FAULT_N) -> MCU-GPIO15
- U1 pad 17: unconnected-(U1-SHD/SD2-Pad17) -> MCU-GPIO9
- U1 pad 18: unconnected-(U1-SWP/SD3-Pad18) -> MCU-GPIO10
- U1 pad 19: unconnected-(U1-SCS/CMD-Pad19) -> MCU-GPIO11
- U5 pad 26: Net-(U5-FAULT_N) -> MCU-GPIO15
Routing:
- net DISPLAY_5V: track 64.5 -> 122.2 mm
- net MCU-GPIO15: track 0.00 -> 32.0 mm, vias 0 -> 2
- net MOTOR_HALL_C: track 0.00 -> 30.6 mm
- net MCU-GPIO11: track 0.00 -> 30.6 mm, vias 0 -> 2
- net MCU-GPIO9: track 0.00 -> 29.1 mm, vias 0 -> 2
- net MCU-GPIO10: track 0.00 -> 28.0 mm, vias 0 -> 2
- net MOTOR_HALL_B: track 0.00 -> 24.8 mm
- net MOTOR_HALL_A: track 0.00 -> 19.0 mm
- net BRAKE_GND: track 23.8 -> 28.8 mm, vias 34 -> 37
- net Net-(U5-FAULT_N): track 4.19 -> 0.00 mm
