File: KiCad/BeanBike/Controller/beanbike_controller_connectors.kicad_sch (KiCad schematic)
At the start: 4 parts, among them J2 Motor Conn, J3 PAS Conn, J4 Throttle Conn, J5 Disp Conn

Commit message: PCB v1
Whole lotta stuff
Parts:
- removed J5: Disp Conn, symbol Connector:Conn_01x05_Pin
- added J5: Display Conn, Connector_PinHeader_2.54mm:PinHeader_1x06_P2.54mm_Vertical, symbol Connector:Conn_01x06_Pin
- added J6: Brake Conn, Connector_PinHeader_2.54mm:PinHeader_1x02_P2.54mm_Vertical, symbol Connector:Conn_01x02_Pin
- J2: footprint (none) -> Connector_PinHeader_2.54mm:PinHeader_1x08_P2.54mm_Vertical
- J3: renamed from J4; footprint (none) -> Connector_PinHeader_2.54mm:PinHeader_1x03_P2.54mm_Vertical
- J4: renamed from J3; footprint (none) -> Connector_PinHeader_2.54mm:PinHeader_1x03_P2.54mm_Vertical
Connections:
- net PAS_GND is gone; now on net GND: J4.2 (Pin_2)
- net THROTTLE_5V is gone; now on net +5V: J3.1 (Pin_1)
- net THROTTLE_GND is gone; now on net GND: J3.2 (Pin_2)
- net MOTOR_HALL_GND renamed GND
- net GND: now also J5.2 (Pin_2), J6.1 (Pin_1)
- net PAS_5V renamed +5V
- net +5V: now also J5.1 (Pin_1)
- net PAS_PULSE renamed MCU-GPIO22
- net THROTTLE_DATA renamed MCU-GPIO21
- new net BRAKE_SIGNAL: J6.2 (Pin_2)
- new net MCU-Boot: J5.6 (Pin_6)
- new net MCU-RX: J5.3 (Pin_3)
- new net MCU-Reset: J5.5 (Pin_5)
- new net MCU-TX: J5.4 (Pin_4)
Other:
- note added: "Brake Connector"

Commit message: PCBv2 Finish
Connections:
- net MCU-GPIO21 renamed MCU-GPIO34
- net MCU-GPIO22 renamed MCU-GPIO35
Changed lines of the file:
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@@
 		)
 	)
-	(global_label "MCU-GPIO21"
+	(global_label "MCU-GPIO34"
 		(shape input)
 		(at 195.58 71.12 0)
@@
 		)
 	)
-	(global_label "MCU-GPIO23"
+	(global_label "MCU-GPIO32"
 		(shape input)
 		(at 195.58 90.17 0)
@@
 		)
 	)
-	(global_label "MCU-GPIO22"
+	(global_label "MCU-GPIO35"
 		(shape input)
 		(at 195.58 81.28 0)

Commit message: More Firmware
😄
Parts:
- added R10, R6, R8: 10k, Resistor_SMD:R_0603_1608Metric, symbol Device:R
- added R11, R7, R9: 18k, Resistor_SMD:R_0603_1608Metric, symbol Device:R
Connections:
- net MOTOR_HALL_5V is gone; now on net +5V: J2.4 (Pin_4)
- net GND: now also R11.2, R7.2, R9.2
- net MOTOR_HALL_A: now also R6.1
- net MOTOR_HALL_B: now also R8.1
- net MOTOR_HALL_C: now also R10.1
- new net MCU-GPIO10: R8.2, R9.1
- new net MCU-GPIO11: R10.2, R11.1
- new net MCU-GPIO9: R6.2, R7.1
