File: PCB/BeanBike/Controller/beanbike_controller.kicad_sch (KiCad schematic)
At the start: 14 parts, among them SW1 SW_SPDT, U4 STM32G473RETx

Commit message: CAN
Parts:
- removed FB1: 600R@100MHz, symbol Device:FerriteBead
- added C14, C15: 30pF, symbol Device:C
- added R16: 0 Ohm (bridge), symbol Device:R
- added X1: X49SM8MSD2SC, easyeda2kicad:CRYSTAL-SMD_L11.5-W4.8-LS12.7, symbol easyeda2kicad:X49SM8MSD2SC
Connections:
- net +3.3V: now also R16.2
- net GND: now also C14.2, C15.2
- net MCU_SPI1_SCK: now reaches U4.19 (PA5)
- net MCU_SPI1_MISO: now reaches U4.20 (PA6)
- net MCU_SPI1_MOSI: now reaches U4.21 (PA7)
- net at U4.29 (VDDA): now also R16.1
- net CAN/CAN_RX: now reaches U4.45 (PA11)
- net CAN/CAN_TX: now reaches U4.46 (PA12)
- net MCU_i2c1_SCL: now reaches U4.49 (PA13)
- net HSE_IN: now reaches U4.5 (PF0)
- net HSE_IN: now also C15.1, X1.2 (OSC2)
- net MCU_i2c1_SDA: now reaches U4.50 (PA14)
- net HSE_OUT: now reaches U4.6 (PF1)
- net HSE_OUT: now also C14.1, X1.1 (OSC1)
Other:
- added sheet CAN (can.kicad_sch)

Commit message: Schematic v3 Done
Parts:
- removed C9: 4.7uF, symbol Device:C
- removed SW1: SW_SPDT, symbol Switch:SW_SPDT
- added SW1: SW_Push, symbol Switch:SW_Push
- C5, C6, C7, C8: value 100nf -> 100nF
Connections:
- net +3.3V: now also C5.2, C6.2, C7.2, C8.2, SW1.2; no longer C5.1, C6.1, C7.1, C8.1
- net GND: now also C5.1, C6.1, C7.1, C8.1; no longer C5.2, C6.2, C7.2, C8.2
- net at R12.2: now also SW1.1
- net MCU_PC2: now reaches U4.10 (PC2)
- net MCU_PC3: now reaches U4.11 (PC3)
- net MCU_SOA: now reaches U4.12 (PA0)
- net MCU_SOB: now reaches U4.13 (PA1)
- net MCU_SOC: now reaches U4.14 (PA2)
- net MCU_PA3: now reaches U4.17 (PA3)
- net MCU_PA4: now reaches U4.18 (PA4)
- net MCU_PC13: now reaches U4.2 (PC13)
- net MCU_PB0: now reaches U4.24 (PB0)
- net MCU_PB1: now reaches U4.25 (PB1)
- net MCU_PB2: now reaches U4.26 (PB2)
- net MCU_PC14: now reaches U4.3 (PC14)
- net MCU_PB10: now reaches U4.30 (PB10)
- net MCU_PB11: now reaches U4.33 (PB11)
- net MCU_PB12: now reaches U4.34 (PB12)
- net MCU_INLA: now reaches U4.35 (PB13)
- net MCU_INLB: now reaches U4.36 (PB14)
- net MCU_INLC: now reaches U4.37 (PB15)
- net MCU_PC6: now reaches U4.38 (PC6)
- net MCU_PC7: now reaches U4.39 (PC7)
- net MCU_PC15: now reaches U4.4 (PC15)
- net MCU_PC8: now reaches U4.40 (PC8)
- net MCU_PC9: now reaches U4.41 (PC9)
- net MCU_INHA: now reaches U4.42 (PA8)
- net MCU_INHB: now reaches U4.43 (PA9)
- net MCU_INHC: now reaches U4.44 (PA10)
- net MCU_PA15: now reaches U4.51 (PA15)
- net MCU_PC10: now reaches U4.52 (PC10)
- net MCU_PC11: now reaches U4.53 (PC11)
- net MCU_PC12: now reaches U4.54 (PC12)
- net MCU_PD2: now reaches U4.55 (PD2)
- net MCU_PB3: now reaches U4.56 (PB3)
- net MCU_PB4: now reaches U4.57 (PB4)
- net MCU_PB5: now reaches U4.58 (PB5)
- net MCU_PB6: now reaches U4.59 (PB6)
- net MCU_PB7: now reaches U4.60 (PB7)
- net MCU_PB9: now reaches U4.62 (PB9)
- net MCU_PC0: now reaches U4.8 (PC0)
- net MCU_PC1: now reaches U4.9 (PC1)

Commit message: Footprints
Parts:
- C10, C12, C13, C5, C6, C7, C8: footprint (none) -> Capacitor_SMD:C_0402_1005Metric; LCSC (none) -> C1525
- C11: footprint (none) -> Capacitor_SMD:C_0402_1005Metric; LCSC (none) -> C52923
- C14, C15: footprint (none) -> Capacitor_SMD:C_0402_1005Metric; LCSC (none) -> C1570
- R12: footprint (none) -> Resistor_SMD:R_0805_2012Metric; LCSC (none) -> C17414
- R13, R16: footprint (none) -> Resistor_SMD:R_0805_2012Metric; LCSC (none) -> C17477
- SW1: footprint (none) -> easyeda2kicad:SW-SMD_L3.9-W3.0-P4.45; LCSC (none) -> C720477
Changed lines of the file:
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@@
 			)
 		)
-		(property "Footprint" ""
+		(property "Footprint" "easyeda2kicad:SW-SMD_L3.9-W3.0-P4.45"
 			(at 207.01 118.11 0)
 			(effects
@@
 			)
 		)
+		(property "LCSC" "C720477"
+			(at 207.01 123.19 0)
+			(effects
+				(font
+					(size 1.27 1.27)
+				)
+				(hide yes)
+			)
+		)
 		(pin "1"
 		)
@@
 			)
 		)
-		(property "Footprint" ""
+		(property "Footprint" "Capacitor_SMD:C_0402_1005Metric"
 			(at 75.2348 41.91 0)
 			(effects
@@
 			)
 		)
+		(property "LCSC" "C1525"
+			(at 76.2 45.72 0)
+			(effects
+				(font
+					(size 1.27 1.27)
+				)
+				(hide yes)
+			)
+		)
 		(pin "1"
 		)
@@
 			)
 		)
-		(property "Footprint" ""
+		(property "Footprint" "Capacitor_SMD:C_0402_1005Metric"
 			(at 114.6048 41.91 0)
 			(effects
@@
 			)
 		)
+		(property "LCSC" "C1525"
+			(at 115.57 45.72 0)
+			(effects
+				(font
+					(size 1.27 1.27)
+				)
+				(hide yes)
+			)
+		)
 		(pin "1"
 		)
@@
 			)
 		)
-		(property "Footprint" ""
+		(property "Footprint" "Resistor_SMD:R_0805_2012Metric"
 			(at 146.558 41.91 90)
 			(effects
@@
 			)
 		)
+		(property "LCSC" "C17477"
+			(at 144.78 41.91 0)
+			(effects
+				(font
+					(size 1.27 1.27)
+				)
+				(hide yes)
+			)
+		)
 		(pin "1"
 		)
@@
 			)
 		)
-		(property "Footprint" ""
+		(property "Footprint" "Capacitor_SMD:C_0402_1005Metric"
 			(at 165.1 150.1648 0)
 			(effects
@@
 			)
 		)
+		(property "LCSC" "C52923"
+			(at 161.29 151.13 90)
+			(effects
+				(font
+					(size 1.27 1.27)
+				)
+				(hide yes)
+			)
+		)
 		(pin "2"
 		)
@@
 			)
 		)
-		(property "Footprint" ""
+		(property "Footprint" "Capacitor_SMD:C_0402_1005Metric"
 			(at 63.1952 102.87 0)
 			(effects
@@
 			)
 		)
+		(property "LCSC" "C1570"
+			(at 62.23 99.06 0)
+			(effects
+				(font
+					(size 1.27 1.27)
+				)
+				(hide yes)
+			)
+		)
 		(pin "1"
 		)
@@
 			)
 		)
-		(property "Footprint" ""
+		(property "Footprint" "Capacitor_SMD:C_0402_1005Metric"
 			(at 87.9348 41.91 0)
 			(effects
@@
 			)
 		)
+		(property "LCSC" "C1525"
+			(at 88.9 45.72 0)
+			(effects
+				(font
+					(size 1.27 1.27)
+				)
+				(hide yes)
+			)
+		)
 		(pin "1"
 		)
@@
 			)
 		)
-		(property "Footprint" ""
+		(property "Footprint" "Resistor_SMD:R_0805_2012Metric"
 			(at 189.23 124.968 90)
 			(effects
@@
 			)
 		)
+		(property "LCSC" "C17414"
+			(at 189.23 123.19 90)
+			(effects
+				(font
+					(size 1.27 1.27)
+				)
+				(hide yes)
+			)
+		)
 		(pin "2"
 		)
@@
 			)
 		)
-		(property "Footprint" ""
+		(property "Footprint" "Capacitor_SMD:C_0402_1005Metric"
 			(at 93.6752 72.39 0)
 			(effects
@@
 			)
 		)
+		(property "LCSC" "C1525"
+			(at 92.71 68.58 0)
+			(effects
+				(font
+					(size 1.27 1.27)
+				)
+				(hide yes)
+			)
+		)
 		(pin "1"
 		)
@@
 			)
 		)
-		(property "Footprint" ""
+		(property "Footprint" "Capacitor_SMD:C_0402_1005Metric"
 			(at 101.9048 41.91 0)
 			(effects
@@
 			)
 		)
+		(property "LCSC" "C1525"
+			(at 102.87 45.72 0)
+			(effects
+				(font
+					(size 1.27 1.27)
+				)
+				(hide yes)
+			)
+		)
 		(pin "1"
 		)
@@
 			)
 		)
-		(property "Footprint" ""
+		(property "Footprint" "Resistor_SMD:R_0805_2012Metric"
 			(at 180.34 156.718 90)
 			(effects
@@
 			)
 		)
+		(property "LCSC" "C17477"
+			(at 180.34 154.94 90)
+			(effects
+				(font
+					(size 1.27 1.27)
+				)
+				(hide yes)
+			)
+		)
 		(pin "1"
 		)
@@
 			)
 		)
-		(property "Footprint" ""
+		(property "Footprint" "Capacitor_SMD:C_0402_1005Metric"
 			(at 73.3552 102.87 0)
 			(effects
@@
 			)
 		)
+		(property "LCSC" "C1570"
+			(at 72.39 99.06 0)
+			(effects
+				(font
+					(size 1.27 1.27)
+				)
+				(hide yes)
+			)
+		)
 		(pin "1"
 		)
@@
 			)
 		)
-		(property "Footprint" ""
+		(property "Footprint" "Capacitor_SMD:C_0402_1005Metric"
 			(at 165.1 161.5948 0)
 			(effects
@@
 			)
 		)
+		(property "LCSC" "C1525"
+			(at 161.29 162.56 90)
+			(effects
+				(font
+					(size 1.27 1.27)
+				)
+				(hide yes)
+			)
+		)
 		(pin "2"
 		)
@@
 			)
 		)
-		(property "Footprint" ""
+		(property "Footprint" "Capacitor_SMD:C_0402_1005Metric"
 			(at 190.1952 162.56 0)
 			(effects
@@
 			(at 189.23 158.75 0)
 			(effects
+				(font
+					(size 1.27 1.27)
+				)
+				(hide yes)
+			)
+		)
+		(property "LCSC" "C1525"
+			(at 189.23 158.75 0)
+			(effects

Commit message: PCB v3
Parts:
- removed R13, R16: 0 Ohm (bridge), Resistor_SMD:R_0805_2012Metric, symbol Device:R
- added C16: 100nf, Capacitor_SMD:C_0402_1005Metric, symbol Device:C
- added C17: 1uF, Capacitor_SMD:C_0402_1005Metric, symbol Device:C
- added C9: 4.7uF, Capacitor_SMD:C_0402_1005Metric, symbol Device:C
- U4: LCSC (none) -> C730120
Connections:
- net VREF is gone; now on net +3.3V: C11.2, C12.2, U4.28 (VREF+)
- net +3.3V: now also U4.29 (VDDA), C16.1, C17.1, C9.1
- net GND: now also C9.2
- net GNDA: now also C16.2, C17.2
- net MCU_PA15: no longer names the net of U4.51 (PA15)
- net MCU_PA3: no longer names the net of U4.17 (PA3)
- net MCU_PB10: no longer names the net of U4.30 (PB10)
- net MCU_PB11: no longer names the net of U4.33 (PB11)
- net MCU_PB12: no longer names the net of U4.34 (PB12)
- net MCU_PB6: no longer names the net of U4.59 (PB6)
- net MCU_PB7: no longer names the net of U4.60 (PB7)
- net MCU_PB9: no longer names the net of U4.62 (PB9)
- net MCU_PC0: no longer names the net of U4.8 (PC0)
- net MCU_PC1: no longer names the net of U4.9 (PC1)
- net MCU_PC10: no longer names the net of U4.52 (PC10)
- net MCU_PC11: no longer names the net of U4.53 (PC11)
- net MCU_PC12: no longer names the net of U4.54 (PC12)
- net MCU_PC13: no longer names the net of U4.2 (PC13)
- net MCU_PC14: no longer names the net of U4.3 (PC14)
- net MCU_PC15: no longer names the net of U4.4 (PC15)
- net MCU_PC2: no longer names the net of U4.10 (PC2)
- net MCU_PC3: no longer names the net of U4.11 (PC3)
- net MCU_PC6: no longer names the net of U4.38 (PC6)
- net MCU_PC7: no longer names the net of U4.39 (PC7)
- net MCU_PD2: no longer names the net of U4.55 (PD2)
- net MCU_i2c1_SCL: no longer names the net of U4.49 (PA13)
- net MCU_i2c1_SDA: no longer names the net of U4.50 (PA14)
- no-connect marks 0 -> 23

Commit message: PCB v3
Connections:
- net MCU_PC2: now reaches U4.10 (PC2)
- net MCU_PC0: now reaches U4.8 (PC0)
- net MCU_PC1: now reaches U4.9 (PC1)
- net MCU_PB2: no longer names the net of U4.26 (PB2)
- net MCU_PB3: no longer names the net of U4.56 (PB3)
- net MCU_PB4: no longer names the net of U4.57 (PB4)
Changed lines of the file:
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@@
 	)
 	(no_connect
-		(at 119.38 82.55)
+		(at 154.94 107.95)
+	)
+	(no_connect
+		(at 154.94 110.49)
 	)
 	(no_connect
@@
 	)
 	(no_connect
-		(at 119.38 87.63)
-	)
-	(no_connect
 		(at 154.94 130.81)
 	)
@@
 	)
 	(no_connect
-		(at 119.38 85.09)
+		(at 154.94 113.03)
 	)
 	(no_connect
@@
 	(wire
 		(pts
+			(xy 107.95 82.55) (xy 119.38 82.55)
+		)
+		(stroke
+			(width 0)
+			(type default)
+		)
+	)
+	(wire
+		(pts
 			(xy 168.91 162.56) (xy 168.91 154.94)
 		)
@@
 	(wire
 		(pts
-			(xy 154.94 110.49) (xy 167.64 110.49)
-		)
-		(stroke
-			(width 0)
-			(type default)
-		)
-	)
-	(wire
-		(pts
 			(xy 154.94 140.97) (xy 167.64 140.97)
 		)
@@
 	(wire
 		(pts
+			(xy 107.95 85.09) (xy 119.38 85.09)
+		)
+		(stroke
+			(width 0)
+			(type default)
+		)
+	)
+	(wire
+		(pts
 			(xy 139.7 151.13) (xy 157.48 151.13)
 		)
@@
 	(wire
 		(pts
+			(xy 107.95 87.63) (xy 119.38 87.63)
+		)
+		(stroke
+			(width 0)
+			(type default)
+		)
+	)
+	(wire
+		(pts
 			(xy 134.62 49.53) (xy 132.08 49.53)
 		)
@@
 	(wire
 		(pts
-			(xy 154.94 107.95) (xy 167.64 107.95)
-		)
-		(stroke
-			(width 0)
-			(type default)
-		)
-	)
-	(wire
-		(pts
 			(xy 88.9 49.53) (xy 102.87 49.53)
 		)
@@
 		(pts
 			(xy 132.08 41.91) (xy 132.08 49.53)
-		)
-		(stroke
-			(width 0)
-			(type default)
-		)
-	)
-	(wire
-		(pts
-			(xy 154.94 113.03) (xy 167.64 113.03)
 		)
 		(stroke
@@
 		)
 	)
-	(global_label "MCU_PB3"
-		(shape input)
-		(at 167.64 110.49 0)
-		(fields_autoplaced yes)
-		(effects
-			(font
-				(size 1.27 1.27)
-			)
-			(justify left)
-		)
-		(property "Intersheetrefs" "${INTERSHEET_REFS}"
-			(at 179.3942 110.49 0)
-			(effects
-				(font
-					(size 1.27 1.27)
-				)
-				(justify left)
-				(hide yes)
-			)
-		)
-	)
 	(global_label "MCU_PC8"
 		(shape input)
@@
 		)
 	)
-	(global_label "MCU_PB4"
-		(shape input)
-		(at 167.64 113.03 0)
-		(fields_autoplaced yes)
-		(effects
-			(font
-				(size 1.27 1.27)
-			)
-			(justify left)
-		)
-		(property "Intersheetrefs" "${INTERSHEET_REFS}"
-			(at 179.3942 113.03 0)
-			(effects
-				(font
-					(size 1.27 1.27)
-				)
-				(justify left)
-				(hide yes)
-			)
-		)
-	)
 	(global_label "MCU_INHC"
 		(shape input)
@@
 		)
 	)
+	(global_label "MCU_PC1"
+		(shape input)
+		(at 107.95 85.09 180)
+		(fields_autoplaced yes)
+		(effects
+			(font
+				(size 1.27 1.27)
+			)
+			(justify right)
+		)
+		(property "Intersheetrefs" "${INTERSHEET_REFS}"
+			(at 96.1958 85.09 0)
+			(effects
+				(font
+					(size 1.27 1.27)
+				)
+				(justify right)
+				(hide yes)
+			)
+		)
+	)
 	(global_label "MCU_PC9"
 		(shape input)
@@
 		)
 	)
-	(global_label "MCU_PB2"
-		(shape input)
-		(at 167.64 107.95 0)
-		(fields_autoplaced yes)
-		(effects
-			(font
-				(size 1.27 1.27)
-			)
-			(justify left)
-		)
-		(property "Intersheetrefs" "${INTERSHEET_REFS}"
-			(at 179.3942 107.95 0)
-			(effects
-				(font
-					(size 1.27 1.27)
-				)
-				(justify left)
-				(hide yes)
-			)
-		)
-	)
 	(global_label "MCU_SOB"
 		(shape input)
@@
 		)
 	)
+	(global_label "MCU_PC0"
+		(shape input)
+		(at 107.95 82.55 180)
+		(fields_autoplaced yes)
+		(effects
+			(font
+				(size 1.27 1.27)
+			)
+			(justify right)
+		)
+		(property "Intersheetrefs" "${INTERSHEET_REFS}"
+			(at 96.1958 82.55 0)
+			(effects
+				(font
+					(size 1.27 1.27)
+				)
+				(justify right)
+				(hide yes)
+			)
+		)
+	)
 	(global_label "MCU_RX"
 		(shape input)
@@
 				(hide yes)
 			)
+		)
+	)
+	(global_label "MCU_PC2"
+		(shape input)
+		(at 107.95 87.63 180)
+		(fields_autoplaced yes)
+		(effects
+			(font
+				(size 1.27 1.27)
+			)
+			(justify right)
+		)
+		(property "Intersheetrefs" "${INTERSHEET_REFS}"
+			(at 96.1958 87.63 0)
+			(effects
+				(font
+					(size 1.27 1.27)
+				)
+				(justify right)
+				(hide yes)
+			)

Commit message: big ol update
Parts:
- added D3: LED, LED_SMD:LED_0805_2012Metric, symbol Device:LED
- added R7: 330, Resistor_SMD:R_0805_2012Metric, symbol Device:R
Connections:
- net +3.3V: now also D3.2 (A)
- net BOOT: now also R12.2, SW1.1; no longer R12.1
- net GND: now also R12.1
- net MCU-LED: now reaches U4.33 (PB11)
- net MCU-LED: now also R7.1
- net MCU_SWDIO: now reaches U4.49 (PA13)
- net MCU_SWCLK: now reaches U4.50 (PA14)
- net MCU_SWO: now reaches U4.56 (PB3)
- new net: D3.1 (K), R7.2
- no-connect marks 23 -> 19
Other:
- moved on the sheet: R12
