File: PCB/BeanBike/Controller/_autosave-beanbike_controller.kicad_sch (KiCad schematic)
At the start: 14 parts, among them SW1 SW_SPDT, U4 STM32G473RETx

Commit message: Fix Spacing and Layout
Parts:
- added C14, C15: 30pF, symbol Device:C
- added X1: X49SM8MSD2SC, easyeda2kicad:CRYSTAL-SMD_L11.5-W4.8-LS12.7, symbol easyeda2kicad:X49SM8MSD2SC
Connections:
- net GND: now also C14.2, C15.2
- net HSE_IN: now reaches U4.5 (PF0)
- net HSE_IN: now also C15.1, X1.2 (OSC2)
- net HSE_OUT: now reaches U4.6 (PF1)
- net HSE_OUT: now also C14.1, X1.1 (OSC1)
