File: PCB/BeanBike/Controller/can.kicad_sch (KiCad schematic)
At the start: 2 parts, among them U1 SN65HVD230DR

Commit message: Footprints
Parts:
- R14: footprint (none) -> Resistor_SMD:R_0805_2012Metric; LCSC (none) -> C17437
Changed lines of the file:
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@@
 			)
 		)
-		(property "Footprint" ""
+		(property "Footprint" "Resistor_SMD:R_0805_2012Metric"
 			(at 216.408 95.25 90)
 			(effects
@@
 			(effects
 				(font
+					(size 1.27 1.27)
+				)
+				(hide yes)
+			)
+		)
+		(property "LCSC" "C17437"
+			(at 214.63 95.25 90)
+			(effects
+				(font
