File: PCB/BeanBike/Controller/Controller.kicad_pcb (KiCad board)
At the start: 6 copper layers, 49.8 x 70.4 mm, 58 parts, among them J1 XT80 Male, J2 Motor Conn, J3 Throttle Conn, J4 PAS Conn, J5 Display Conn, J6 Brake Conn, Q1 PHASE A HIGH, Q2 PHASE B HIGH, Q3 PHASE C HIGH, Q4 PHASE A LOW, Q5 PHASE B LOW, Q6 PHASE C LOW, U1 ESP32-WROOM-32, U5 DRV8353SRTAT

Commit message: Footprints
Parts:
- removed C16: 100nf, Capacitor_SMD:C_0201_0603Metric
- removed C17: 22uF, Capacitor_SMD:C_0603_1608Metric
- removed C9: 100nF, Capacitor_SMD:C_0201_0603Metric
- removed F1: Fuse, Fuse:Fuse_1206_3216Metric
- removed L2: L, easyeda2kicad:IND-SMD_L4.8-W4.5
- removed PS1, PS2: LMR38025SQDRRRQ1, LMR380:SON50P300X300X80-13N
- removed R17: 46.4k, Resistor_SMD:R_0402_1005Metric
- removed R18, R20, R22, R24: 10k, Resistor_SMD:R_0603_1608Metric
- removed R19: 40.2k, Resistor_SMD:R_0402_1005Metric
- removed R21: 21.5k, Resistor_SMD:R_0402_1005Metric
- removed R23: 23.2k, Resistor_SMD:R_0402_1005Metric
- added C1: 680uF 63V, Capacitor_THT:CP_Radial_D12.5mm_P5.00mm, F.Cu at (137.4, 67.5)
- added C2: 330uF 25V, Capacitor_THT:CP_Radial_D8.0mm_P3.50mm, F.Cu at (152.8, 53.5)
- added C3: 22uF, Capacitor_SMD:C_0201_0603Metric, F.Cu at (167.1, 68.0)
- added C4: 10uf, Capacitor_SMD:C_0402_1005Metric, F.Cu at (164.5, 68.1)
- added C5: 100nF, Capacitor_SMD:C_0402_1005Metric, F.Cu at (172.1, 78.2)
- added C6: 100nF, Capacitor_SMD:C_0402_1005Metric, F.Cu at (172.1, 80.1)
- added D1: D, Diode_SMD:D_SOD-123F, F.Cu at (149.7, 73.5)
- added J7: DEBUG Conn, Connector_PinHeader_2.54mm:PinHeader_1x03_P2.54mm_Vertical, F.Cu at (151.9, 97.2)
- added R12: 10k, Resistor_SMD:R_0805_2012Metric, F.Cu at (158.4, 93.1)
- added R13: 0 Ohm (bridge), Resistor_SMD:R_0805_2012Metric, F.Cu at (158.4, 96.0)
- added R14: 120, Resistor_SMD:R_0805_2012Metric, F.Cu at (171.8, 50.1)
- added R16: 0 Ohm (bridge), Resistor_SMD:R_0805_2012Metric, F.Cu at (158.4, 99.0)
- added SW1: SW_Push, easyeda2kicad:SW-SMD_L3.9-W3.0-P4.45, F.Cu at (173.9, 89.1)
- added U2: TD1501HS50, easyeda2kicad:PG-TO-263-5_L10.2-W8.7-P1.70-LS14.4-BR, F.Cu at (142.1, 54.6)
- added U3: AMS1117-3.3, easyeda2kicad:SOT-223-3_L6.5-W3.4-P2.30-LS7.0-BR, F.Cu at (167.7, 63.2)
- added U4: STM32G473RETx, Package_QFP:LQFP-64_10x10mm_P0.5mm, F.Cu at (163.4, 84.4)
- added X1: X49SM8MSD2SC, easyeda2kicad:CRYSTAL-SMD_L11.5-W4.8-LS12.7, F.Cu at (168.3, 94.7)
- C10, C18, C20, C22, C23, C24: footprint Capacitor_SMD:C_0201_0603Metric -> Capacitor_SMD:C_0402_1005Metric
- C11: value 22uF -> 1uF; footprint Capacitor_SMD:C_0603_1608Metric -> Capacitor_SMD:C_0402_1005Metric
- C12: value 22uF -> 100nf; footprint Capacitor_SMD:C_0603_1608Metric -> Capacitor_SMD:C_0402_1005Metric
- C13: value 2.2uF -> 100nf; footprint Capacitor_SMD:C_0201_0603Metric -> Capacitor_SMD:C_0402_1005Metric
- C14: value 2.2uF -> 30pF; footprint Capacitor_SMD:C_0201_0603Metric -> Capacitor_SMD:C_0402_1005Metric
- C15: value 100nF -> 30pF; footprint Capacitor_SMD:C_0201_0603Metric -> Capacitor_SMD:C_0402_1005Metric
- C19: footprint Capacitor_SMD:C_0603_1608Metric -> Capacitor_SMD:C_0805_2012Metric
- C21: footprint Capacitor_SMD:C_0201_0603Metric -> Capacitor_SMD:C_0603_1608Metric
- C7, C8: value 2.2uF -> 100nF; footprint Capacitor_SMD:C_0201_0603Metric -> Capacitor_SMD:C_0402_1005Metric
- J1: footprint Connector_Wire:SolderWire-2sqmm_1x02_P7.8mm_D2mm_OD3.9mm -> XT60PW-M:AMASS_XT60PW-M
- L1: value 8.2uH 68mOhm -> CYA1040-33UH; footprint easyeda2kicad:IND-SMD_L7.1-W6.6 -> easyeda2kicad:IND-SMD_L11.6-W10.1
- Q1, Q2, Q3, Q4, Q5, Q6: footprint Package_TO_SOT_THT:TO-220-3_Vertical -> TO-220AB:TO254P1050X476X2020-3
- R1, R10, R11, R2, R25, R26, R6, R7, R8, R9: footprint Resistor_SMD:R_0603_1608Metric -> Resistor_SMD:R_0805_2012Metric
- R3, R4, R5: footprint Resistor_SMD:R_2512_6332Metric -> footprints:RES_1L00x_BRN
- U1: value ESP32-WROOM-32 -> SN65HVD230DR; footprint RF_Module:ESP32-WROOM-32 -> easyeda2kicad:SOIC-8_L4.9-W3.9-P1.27-LS6.0-BL
- U5: footprint MOTORIC:RTA0040B -> DRV8353:QFN50P600X600X80-41N
- moved C7 77.4 mm to (172.1, 82.1)
- moved C8 75.3 mm to (172.1, 84.1)
- moved L1 75.2 mm to (154.0, 66.2)
- moved C11 71.2 mm to (174.9, 78.2), turned to 0 degrees
- moved C12 71.0 mm to (174.9, 80.1), turned to 0 degrees
- moved C10 69.1 mm to (172.1, 86.0), turned to 0 degrees
- moved Q1 66.4 mm to (115.6, 51.7)
- moved C13 66.2 mm to (174.9, 82.1), turned to 0 degrees
- moved C14 64.3 mm to (174.9, 84.1), turned to 0 degrees
- moved C15 62.5 mm to (174.9, 86.0), turned to 0 degrees
- moved R3 60.6 mm to (125.9, 51.1)
- moved Q2 57.9 mm to (115.6, 57.9)
- moved J6 52.9 mm to (151.7, 79.5)
- moved R4 52.3 mm to (125.9, 56.0)
- moved Q3 50.9 mm to (115.6, 64.0)
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Connections:
- C10 pad 1: Net-(PS1-BOOT) -> +3.3V
- C10 pad 2: Net-(PS1-SW_1) -> GNDA
- C11 pad 1: BRAKE_GND -> GNDA
- C11 pad 2: DISPLAY_5V -> /MCU/VREF
- C12 pad 1: BRAKE_GND -> GNDA
- C12 pad 2: DISPLAY_5V -> /MCU/VREF
- C13 pad 1: DISPLAY_5V -> RST
- C14 pad 1: DISPLAY_5V -> /MCU/HSE_OUT
- C15 pad 1: DISPLAY_5V -> /MCU/HSE_IN
- C20 pad 2: /Motor/VDRAIN -> PWR_MOTOR
- C7 pad 1: PWR_MOTOR -> BRAKE_GND
- C7 pad 2: BRAKE_GND -> +3.3V
- C8 pad 1: PWR_MOTOR -> BRAKE_GND
- C8 pad 2: BRAKE_GND -> +3.3V
- J1 pad 1: +BATT -> PWR_MOTOR
- L1 pad 1: Net-(PS1-SW_1) -> Net-(D1-K)
- Q4 pad 2: BRAKE_GND -> MOTOR_PHASE_A
- Q4 pad 3: MOTOR_PHASE_A -> Net-(Q4-S)
- Q5 pad 2: BRAKE_GND -> MOTOR_PHASE_B
- Q5 pad 3: MOTOR_PHASE_B -> Net-(Q5-S)
- Q6 pad 2: BRAKE_GND -> MOTOR_PHASE_C
- Q6 pad 3: MOTOR_PHASE_C -> Net-(Q6-S)
- R25 pad 1: MCU-GPIO19 -> MCU_SPI1_MOSI
- R26 pad 2: MCU-GPIO15 -> MCU_PC8
- R3 pad 1: MOTOR_PHASE_C -> Net-(Q6-S)
- R4 pad 1: MOTOR_PHASE_B -> Net-(Q5-S)
- R5 pad 1: MOTOR_PHASE_A -> Net-(Q4-S)
- U1 pad 1: BRAKE_GND -> /MCU/CAN/CAN_TX
- U1 pad 2: +3.3V -> BRAKE_GND
- U1 pad 3: MCU-Reset -> +3.3V
- U1 pad 4: unconnected-(U1-SENSOR_VP-Pad4) -> /MCU/CAN/CAN_RX
- U1 pad 6: MCU-GPIO34 -> MCU_CAN-
- U1 pad 7: MCU-GPIO35 -> MCU_CAN+
- U1 pad 8: BRAKE_SIGNAL -> BRAKE_GND
- U5 pad 12: MOTOR_PHASE_B -> Net-(Q5-S)
- U5 pad 19: MOTOR_PHASE_C -> Net-(Q6-S)
- U5 pad 21: MCU-GPIO17 -> MCU_SOC
- U5 pad 22: MCU-GPIO22 -> MCU_SOB
- U5 pad 23: MCU-GPIO21 -> MCU_SOA
- U5 pad 26: MCU-GPIO15 -> MCU_PC8
- U5 pad 27: MCU-GPIO19 -> MCU_SPI1_MOSI
- U5 pad 28: MCU-GPIO23 -> MCU_SPI1_MISO
- U5 pad 29: MCU-GPIO18 -> MCU_SPI1_SCK
- U5 pad 30: MCU-GPIO5 -> MCU_PA4
- U5 pad 31: MCU-GPIO13 -> MCU_PC9
- U5 pad 32: MCU-GPIO12 -> MCU_INHA
- U5 pad 33: MCU-GPIO14 -> MCU_INLA
- U5 pad 34: MCU-GPIO27 -> MCU_INHB
- U5 pad 35: MCU-GPIO26 -> MCU_INLB
- U5 pad 36: MCU-GPIO25 -> MCU_INHC
- U5 pad 37: MCU-GPIO33 -> MCU_INLC
- U5 pad 4: /Motor/VDRAIN -> PWR_MOTOR
- U5 pad 9: MOTOR_PHASE_A -> Net-(Q4-S)
Routing:
- net DISPLAY_5V: track 121.1 -> 0.00 mm
- net +3.3V: track 77.4 -> 0.00 mm
- net BATT_Level: track 67.5 -> 0.00 mm, vias 2 -> 0
- net MCU-GPIO18: track 53.1 -> 0.00 mm, vias 2 -> 0
- net MCU-GPIO19: track 52.0 -> 0.00 mm, vias 2 -> 0
- net MCU-GPIO33: track 46.8 -> 0.00 mm, vias 2 -> 0
- net MCU-GPIO23: track 42.1 -> 0.00 mm, vias 2 -> 0
- net MCU-GPIO25: track 40.8 -> 0.00 mm, vias 2 -> 0
- net MCU-Boot: track 40.0 -> 0.00 mm
- net MCU-GPIO22: track 38.7 -> 0.00 mm, vias 2 -> 0
- net BRAKE_SIGNAL: track 36.5 -> 0.00 mm, vias 1 -> 0
- net MCU-GPIO26: track 34.3 -> 0.00 mm, vias 2 -> 0
- net MCU-GPIO17: track 33.1 -> 0.00 mm, vias 3 -> 0
- net MCU-GPIO5: track 32.5 -> 0.00 mm, vias 2 -> 0
- net MCU-GPIO14: track 32.1 -> 0.00 mm, vias 2 -> 0
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- removed copper zone on B.Cu, net BRAKE_GND
- removed copper zone on In3.Cu, net MOTOR_PHASE_A
- removed copper zone on In2.Cu, net MOTOR_PHASE_B
- removed copper zone on In1.Cu, net MOTOR_PHASE_C
- removed copper zone on In4.Cu, net PWR_MOTOR
Other:
- board outline removed
- board text removed: "Bean Bike"
- board text removed: "BeanBike Controller 48v 1200w"
- board text removed: "GINOBEANO"

Commit message: PCB v3
Parts:
- removed R10, R6, R8: 10k, Resistor_SMD:R_0805_2012Metric
- removed R11, R7, R9: 18k, Resistor_SMD:R_0805_2012Metric
- removed R13, R16: 0 Ohm (bridge), Resistor_SMD:R_0805_2012Metric
- added C16: 100nf, Capacitor_SMD:C_0402_1005Metric, F.Cu at (209.6, 80.4)
- added C17: 1uF, Capacitor_SMD:C_0402_1005Metric, F.Cu at (210.6, 80.4)
- added C9: 4.7uF, Capacitor_SMD:C_0402_1005Metric, F.Cu at (207.6, 94.9)
- added U6: SN74LVC4245APWR, easyeda2kicad:TSSOP-24_L7.8-W4.4-P0.65-LS6.4-BL, F.Cu at (153.3, 82.2)
- moved Q6 153.1 mm to (249.8, 156.2), turned to 180 degrees
- moved Q5 144.8 mm to (236.4, 156.2), turned to 180 degrees
- moved Q4 137.6 mm to (223.0, 156.2), turned to 180 degrees
- moved Q3 131.6 mm to (209.6, 156.2), turned to 180 degrees
- moved Q2 127.1 mm to (196.2, 156.2), turned to 180 degrees
- moved R3 126.5 mm to (214.7, 141.2), turned to -90 degrees
- moved Q1 124.2 mm to (182.8, 156.2), turned to 180 degrees
- moved R4 119.5 mm to (209.8, 141.2), turned to -90 degrees
- moved C4 115.6 mm to (278.8, 50.7)
- moved J5 114.3 mm to (261.3, 75.3)
- moved R5 112.6 mm to (204.9, 141.2), turned to -90 degrees
- moved C3 112.6 mm to (278.8, 53.7)
- moved C24 108.9 mm to (215.5, 129.7)
- moved R25 108.6 mm to (216.3, 126.2)
- moved R26 108.1 mm to (216.3, 128.2), turned to 180 degrees
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- renumbered SW1 to BOOT
Connections:
- C11 pad 2: /MCU/VREF -> +3.3V
- C12 pad 2: /MCU/VREF -> +3.3V
- J3 pad 3: MCU-GPIO34 -> THROTTLE_DATA
- J4 pad 3: MCU-GPIO35 -> PAS_PULSE
- J5 pad 3: MCU-RX -> MCU_CAN+
- J5 pad 4: MCU-TX -> MCU_CAN-
- J5 pad 5: MCU-Reset -> RST
- J5 pad 6: MCU-Boot -> BOOT
- U4 pad 10: MCU_PC2 -> unconnected-(U4-PC2-Pad10)
- U4 pad 11: MCU_PC3 -> unconnected-(U4-PC3-Pad11)
- U4 pad 17: MCU_PA3 -> unconnected-(U4-PA3-Pad17)
- U4 pad 2: MCU_PC13 -> unconnected-(U4-PC13-Pad2)
- U4 pad 28: /MCU/VREF -> +3.3V
- U4 pad 29: Net-(U4-VDDA) -> +3.3V
- U4 pad 3: MCU_PC14 -> unconnected-(U4-PC14-Pad3)
- U4 pad 30: MCU_PB10 -> unconnected-(U4-PB10-Pad30)
- U4 pad 33: MCU_PB11 -> unconnected-(U4-PB11-Pad33)
- U4 pad 34: MCU_PB12 -> unconnected-(U4-PB12-Pad34)
- U4 pad 38: MCU_PC6 -> unconnected-(U4-PC6-Pad38)
- U4 pad 39: MCU_PC7 -> unconnected-(U4-PC7-Pad39)
- U4 pad 4: MCU_PC15 -> unconnected-(U4-PC15-Pad4)
- U4 pad 49: MCU_i2c1_SCL -> unconnected-(U4-PA13-Pad49)
- U4 pad 50: MCU_i2c1_SDA -> unconnected-(U4-PA14-Pad50)
- U4 pad 51: MCU_PA15 -> unconnected-(U4-PA15-Pad51)
- U4 pad 52: MCU_PC10 -> unconnected-(U4-PC10-Pad52)
- U4 pad 53: MCU_PC11 -> unconnected-(U4-PC11-Pad53)
- U4 pad 54: MCU_PC12 -> unconnected-(U4-PC12-Pad54)
- U4 pad 55: MCU_PD2 -> unconnected-(U4-PD2-Pad55)
- U4 pad 58: MCU_PB5 -> BRAKE_SIGNAL
- U4 pad 59: MCU_PB6 -> unconnected-(U4-PB6-Pad59)
- U4 pad 60: MCU_PB7 -> unconnected-(U4-PB7-Pad60)
- U4 pad 62: MCU_PB9 -> unconnected-(U4-PB9-Pad62)
- U4 pad 8: MCU_PC0 -> unconnected-(U4-PC0-Pad8)
- U4 pad 9: MCU_PC1 -> unconnected-(U4-PC1-Pad9)
Routing:
- net +3.3V: track 0.00 -> 30.6 mm
- net PAS_PULSE: track 0.00 -> 23.5 mm
- net MOTOR_HALL_A: track 0.00 -> 20.2 mm
- net MOTOR_HALL_B: track 0.00 -> 19.4 mm
- net MOTOR_HALL_C: track 0.00 -> 18.6 mm
- net THROTTLE_DATA: track 0.00 -> 17.3 mm
- net /MCU/HSE_OUT: track 0.00 -> 17.1 mm
- net /MCU/HSE_IN: track 0.00 -> 15.8 mm
- net MCU_CAN-: track 0.00 -> 11.9 mm
- net MCU_CAN+: track 0.00 -> 11.6 mm
- net BOOT: track 0.00 -> 7.32 mm
- net GNDA: track 0.00 -> 6.20 mm
- net Net-(U5-VM): track 0.00 -> 5.13 mm
- net Net-(U5-CPL): track 0.00 -> 5.02 mm
- net Net-(U5-CPH): track 0.00 -> 4.59 mm
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Other:
- copper layers 6 -> 4

Commit message: PCB v3
Parts:
- added J10: PHASE C, 8196:KEYSTONE_8196, F.Cu at (174.3, 35.2)
- added J8: PHASE A, 8196:KEYSTONE_8196, F.Cu at (217.8, 35.2)
- added J9: PHASE B, 8196:KEYSTONE_8196, F.Cu at (196.1, 35.2)
- J2: value Motor Conn -> Conn_01x05_Pin; footprint Connector_PinHeader_2.54mm:PinHeader_1x08_P2.54mm_Vertical -> Connector_PinHeader_2.54mm:PinHeader_1x05_P2.54mm_Vertical
- moved Q6 138.5 mm to (166.7, 45.5), turned to 0 degrees
- moved Q1 118.2 mm to (224.2, 45.5), turned to 0 degrees
- moved Q5 116.2 mm to (201.2, 45.5), turned to 0 degrees
- moved Q3 115.1 mm to (178.2, 45.5), turned to 0 degrees
- moved Q4 111.2 mm to (212.7, 45.5), turned to 0 degrees
- moved Q2 110.9 mm to (189.7, 45.5), turned to 0 degrees
- moved R3 102.7 mm to (166.7, 50.5), turned to 180 degrees
- moved R5 91.3 mm to (215.2, 50.5), turned to 180 degrees
- moved R4 91.2 mm to (201.2, 50.5), turned to 180 degrees
- moved J1 78.5 mm to (162.8, 63.7), turned to 90 degrees
- moved C24 76.2 mm to (178.0, 63.5), turned to 180 degrees
- moved J7 74.6 mm to (206.8, 125.2), turned to 90 degrees
- moved R26 74.4 mm to (177.2, 65.0), turned to 0 degrees
- moved J2 74.3 mm to (164.1, 125.2), turned to 90 degrees
- moved R25 71.0 mm to (177.2, 67.0), turned to 180 degrees
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- renumbered BOOT to SW1
Connections:
- J2 pad 1: MOTOR_PHASE_A -> DISPLAY_5V
- J2 pad 2: MOTOR_PHASE_B -> BRAKE_GND
- J2 pad 3: MOTOR_PHASE_C -> MOTOR_HALL_A
- J2 pad 4: DISPLAY_5V -> MOTOR_HALL_B
- J2 pad 5: BRAKE_GND -> MOTOR_HALL_C
- U4 pad 10: unconnected-(U4-PC2-Pad10) -> MCU_PC2
- U4 pad 26: MCU_PB2 -> unconnected-(U4-PB2-Pad26)
- U4 pad 56: MCU_PB3 -> unconnected-(U4-PB3-Pad56)
- U4 pad 57: MCU_PB4 -> unconnected-(U4-PB4-Pad57)
- U4 pad 8: unconnected-(U4-PC0-Pad8) -> MCU_PC0
- U4 pad 9: unconnected-(U4-PC1-Pad9) -> MCU_PC1
- U6 pad 19: MCU_PB4 -> MCU_PC2
- U6 pad 20: MCU_PB3 -> MCU_PC1
- U6 pad 21: MCU_PB2 -> MCU_PC0
Routing:
- net DISPLAY_5V: track 3.84 -> 207.1 mm, vias 0 -> 7
- net +3.3V: track 30.6 -> 204.4 mm, vias 0 -> 11
- net BRAKE_GND: track 0.00 -> 79.2 mm, vias 0 -> 60
- net RST: track 4.30 -> 69.1 mm, vias 0 -> 2
- net MCU_SOC: track 0.00 -> 62.3 mm
- net MCU_SOB: track 0.00 -> 61.6 mm
- net MCU_SOA: track 0.00 -> 60.8 mm
- net BOOT: track 7.32 -> 65.3 mm, vias 0 -> 2
- net MCU_SPI1_MISO: track 0.00 -> 50.2 mm, vias 0 -> 2
- net MCU_PC8: track 3.67 -> 52.8 mm, vias 0 -> 2
- net MCU_SPI1_MOSI: track 3.25 -> 50.1 mm, vias 0 -> 2
- net MCU_SPI1_SCK: track 0.00 -> 46.8 mm, vias 0 -> 2
- net BRAKE_SIGNAL: track 0.00 -> 46.1 mm, vias 0 -> 2
- net BLDC-IC_PHASE_A_HIGH: track 0.00 -> 45.7 mm
- net Net-(Q4-S): track 0.00 -> 44.1 mm, vias 0 -> 2
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- added copper zone on In1.Cu, net BRAKE_GND
- added copper zone on In2.Cu, net MOTOR_PHASE_A
- added copper zone on In2.Cu, net MOTOR_PHASE_B
- added copper zone on In2.Cu, net MOTOR_PHASE_C
- added copper zone on In2.Cu, net PWR_MOTOR
Other:
- board outline added: 73.6 x 99.3 mm
- board text added: "BAT_IN"
- board text added: "BEAN BIKE"
- board text added: "BeanBike Controller 48V"
- board text added: "Giovanni Antenucci"
- board text added: "Phase A"
- board text added: "Phase B"
- board text added: "Phase C"
- board text added: "WARNING HIGH CURRENT"

Commit message: big ol update
Parts:
- added D10: 3.3v Zener, Diode_SMD:D_SMA, F.Cu at (216.8, 102.7)
- added D2: LED, LED_SMD:LED_0603_1608Metric, F.Cu at (176.3, 56.7)
- added D3: LED, LED_SMD:LED_0805_2012Metric, F.Cu at (211.3, 99.7)
- added D4: LED, LED_SMD:LED_0603_1608Metric, F.Cu at (227.8, 39.2)
- added D5: LED, LED_SMD:LED_0603_1608Metric, F.Cu at (205.3, 39.2)
- added D6: LED, LED_SMD:LED_0603_1608Metric, F.Cu at (161.8, 37.2)
- added D7: LED, LED_SMD:LED_0603_1608Metric, F.Cu at (227.8, 74.2)
- added D8: LED, LED_SMD:LED_0603_1608Metric, F.Cu at (214.3, 87.2)
- added D9: 5v Zener, Diode_SMD:D_SMA, F.Cu at (213.8, 81.2)
- added F1: 5v Polyfuse, RKEF300:FUS_RKEF300_TYCO_TYC, F.Cu at (204.8, 72.2)
- added F2: 3.3v Polyfuse, MF_R065_2:FUSE_MF_R065_2_BRN, F.Cu at (222.5, 101.1)
- added J11: XT60 -, MountingHole:MountingHole_3.2mm_M3_Pad_Via, F.Cu at (163.3, 73.5)
- added R10: 15k, Resistor_SMD:R_0805_2012Metric, F.Cu at (161.8, 41.7)
- added R11: 1k, Resistor_SMD:R_0805_2012Metric, F.Cu at (227.8, 71.2)
- added R13: 1k, Resistor_SMD:R_0805_2012Metric, F.Cu at (217.3, 87.2)
- added R6: 15k, Resistor_SMD:R_0805_2012Metric, F.Cu at (176.3, 59.7)
- added R7: 330, Resistor_SMD:R_0805_2012Metric, F.Cu at (211.3, 97.7)
- added R8: 15k, Resistor_SMD:R_0805_2012Metric, F.Cu at (227.8, 41.7)
- added R9: 15k, Resistor_SMD:R_0805_2012Metric, F.Cu at (205.3, 41.7)
- J1: value XT80 Male -> XT60 +; footprint XT60PW-M:AMASS_XT60PW-M -> MountingHole:MountingHole_3.2mm_M3_Pad_Via
- J7: value DEBUG Conn -> ST-Link-Debug; footprint Connector_PinHeader_2.54mm:PinHeader_1x03_P2.54mm_Vertical -> Connector_PinHeader_2.54mm:PinHeader_1x06_P2.54mm_Vertical
- moved J7 6.62 mm to (213.4, 125.2), turned to -90 degrees
- moved C1 6.50 mm to (163.8, 87.2)
- moved J3 4.79 mm to (174.3, 125.2)
- moved J4 4.79 mm to (184.4, 125.2)
- moved J6 4.79 mm to (194.5, 125.2)
- moved J2 4.79 mm to (159.4, 125.2)
- moved J1 2.55 mm to (163.3, 61.2), turned to 0 degrees
- moved C2 2.06 mm to (214.5, 72.7)
- moved J5 0.63 mm to (229.8, 125.2)
Connections:
- C18 pad 1: Net-(U5-VM) -> PWR_MOTOR
- C19 pad 1: Net-(U5-VM) -> PWR_MOTOR
- C2 pad 1: DISPLAY_5V -> Net-(U2-FEEDBACK)
- C3 pad 1: +3.3V -> Net-(C3-Pad1)
- J7 pad 1: MCU_TX -> +3.3V
- J7 pad 2: MCU_RX -> MCU_SWDIO
- J7 pad 3: BRAKE_GND -> MCU_SWCLK
- L1 pad 2: DISPLAY_5V -> Net-(U2-FEEDBACK)
- R12 pad 1: BOOT -> BRAKE_GND
- R12 pad 2: Net-(R12-Pad2) -> BOOT
- SW1 pad 1: Net-(R12-Pad2) -> BOOT
- U2 pad 4: DISPLAY_5V -> Net-(U2-FEEDBACK)
- U3 pad 2: +3.3V -> Net-(C3-Pad1)
- U3 pad 4: +3.3V -> Net-(C3-Pad1)
- U4 pad 33: unconnected-(U4-PB11-Pad33) -> MCU-LED
- U4 pad 49: unconnected-(U4-PA13-Pad49) -> MCU_SWDIO
- U4 pad 50: unconnected-(U4-PA14-Pad50) -> MCU_SWCLK
- U4 pad 56: unconnected-(U4-PB3-Pad56) -> MCU_SWO
- U5 pad 3: Net-(U5-VM) -> PWR_MOTOR
Routing:
- net BRAKE_GND: track 79.2 -> 153.0 mm, vias 60 -> 65
- net MCU_SWO: track 0.00 -> 53.6 mm, vias 0 -> 1
- net MCU_SWCLK: track 0.00 -> 53.1 mm, vias 0 -> 1
- net MCU_SWDIO: track 0.00 -> 52.1 mm, vias 0 -> 1
- net MCU_RX: track 36.0 -> 0.00 mm
- net MCU_TX: track 35.2 -> 0.00 mm
- net Net-(U2-FEEDBACK): track 0.00 -> 27.2 mm, vias 0 -> 1
- net PWR_MOTOR: track 38.6 -> 60.9 mm
- net +3.3V: track 204.4 -> 226.0 mm, vias 11 -> 12
- net DISPLAY_5V: track 207.1 -> 187.0 mm, vias 7 -> 10
- net Net-(C3-Pad1): track 0.00 -> 16.1 mm
- net MCU-LED: track 0.00 -> 8.25 mm
- net MOTOR_PHASE_C: track 18.2 -> 25.0 mm
- net Net-(U5-VM): track 5.13 -> 0.00 mm
- net MOTOR_HALL_A: track 20.2 -> 25.1 mm
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Other:
- board size 73.6 x 99.3 mm -> 74.1 x 99.3 mm
- board text added: "- BAT_IN +"
- board text removed: "BAT_IN"
