File: PCB/BeanBike/Controller/Controller.kicad_sch (KiCad schematic)
At the start: 0 parts

Commit message: PCB v3
Changed lines of the file:
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@@
 		(company "Ginobeano")
+	)
+	(symbol
+		(lib_id "Graphic:SYM_Hot_Large")
+		(at 132.08 50.8 0)
+		(unit 1)
+		(exclude_from_sim no)
+		(in_bom yes)
+		(on_board no)
+		(dnp no)
+		(fields_autoplaced yes)
+		(property "Reference" "#SYM1"
+			(at 132.08 45.72 0)
+			(effects
+				(font
+					(size 1.27 1.27)
+				)
+				(hide yes)
+			)
+		)
+		(property "Value" "SYM_Hot_Large"
+			(at 132.08 57.15 0)
+			(effects
+				(font
+					(size 1.27 1.27)
+				)
+				(hide yes)
+			)
+		)
+		(property "Footprint" ""
+			(at 132.08 55.88 0)
+			(effects
+				(font
+					(size 1.27 1.27)
+				)
+				(hide yes)
+			)
+		)
+		(property "Datasheet" "~"
+			(at 132.842 55.88 0)
+			(effects
+				(font
+					(size 1.27 1.27)
+				)
+				(hide yes)
+			)
+		)
+		(property "Description" "Hot surface warning symbol, large"
+			(at 132.08 50.8 0)
+			(effects
+				(font
+					(size 1.27 1.27)
+				)
+				(hide yes)
+			)
+		)
+		(property "Sim.Enable" "0"
+			(at 132.08 50.8 0)
+			(effects
+				(font
+					(size 1.27 1.27)
+				)
+				(hide yes)
+			)
+		)
+		(instances
+			(project ""
+				(path "/645e8d68-d9e1-48b3-98a5-3b81aa58d1ea"
+					(reference "#SYM1")
+					(unit 1)
+				)
+			)
+		)
 	)
 	(sheet

Commit message: big ol update
Other:
- note added: "TODO: SOlid fill vias for thermal grid vias for thermal seprate MOSFETs and Terminals"
Changed lines of the file:
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@@
 		(company "Ginobeano")
+	)
+	(text "TODO:\n\nSOlid fill vias for thermal\ngrid vias for thermal \nseprate MOSFETs and Terminals"
+		(exclude_from_sim no)
+		(at 131.826 91.694 0)
+		(effects
+			(font
+				(size 1.27 1.27)
+			)
+		)
 	)
 	(symbol
@@
 		(at 132.08 50.8 0)
 		(unit 1)
-		(exclude_from_sim no)
+		(exclude_from_sim yes)
 		(in_bom yes)
 		(on_board no)
@@
 			(at 132.08 50.8 0)
 			(effects
-				(font
-					(size 1.27 1.27)
-				)
-				(hide yes)
-			)
-		)
-		(property "Sim.Enable" "0"
-			(at 132.08 50.8 0)
-			(effects
