File: PCB/BeanBike/Controller/beanbike_controller_5v.kicad_sch (KiCad schematic)
At the start: 12 parts

Commit message: Forgot to commit
Parts:
- removed C10: 100nf, Capacitor_SMD:C_0201_0603Metric, symbol Device:C
- removed C11, C12: 22uF, Capacitor_SMD:C_0603_1608Metric, symbol Device:C
- removed C7, C8: 2.2uF, Capacitor_SMD:C_0201_0603Metric, symbol Device:C
- removed C9: 100nF, Capacitor_SMD:C_0201_0603Metric, symbol Device:C
- removed L1: 8.2uH 68mOhm, easyeda2kicad:IND-SMD_L7.1-W6.6, symbol Device:L
- removed PS1: LMR38025SQDRRRQ1, LMR380:SON50P300X300X80-13N, symbol LMR38025SQDRRRQ1:LMR38025SQDRRRQ1
- removed R17: 46.4k, Resistor_SMD:R_0402_1005Metric, symbol Device:R
- removed R18, R20: 10k, Resistor_SMD:R_0603_1608Metric, symbol Device:R
- removed R19: 40.2k, Resistor_SMD:R_0402_1005Metric, symbol Device:R
- added C1: 680uF 63V, symbol Device:C
- added C2: 330uF 25V, symbol Device:C
- added D1: D, symbol Device:D
- added L1: CYA1040-33UH, easyeda2kicad:IND-SMD_L11.6-W10.1, symbol easyeda2kicad:CYA1040-33UH
- added U2: TD1501HS50, easyeda2kicad:PG-TO-263-5_L10.2-W8.7-P1.70-LS14.4-BR, symbol easyeda2kicad:TD1501HS50
Connections:
- net +5V: now also C2.1, L1.2, U2.4 (FEEDBACK)
- net BATT: now also C1.1, U2.1 (VIN)
- net GND: now also C1.2, C2.2, D1.2 (A), U2.3 (GND), U2.5 (ON/OFF), U2.6 (EP)
- new net: D1.1 (K), L1.1, U2.2 (OUTPUT)

Commit message: Footprints
Parts:
- C1: footprint (none) -> Capacitor_THT:CP_Radial_D12.5mm_P5.00mm
- C2: footprint (none) -> Capacitor_THT:CP_Radial_D8.0mm_P3.50mm
- D1: footprint (none) -> Diode_SMD:D_SOD-123F; LCSC (none) -> C64898
Changed lines of the file:
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@@
 			)
 		)
-		(property "Footprint" ""
+		(property "Footprint" "Capacitor_THT:CP_Radial_D8.0mm_P3.50mm"
 			(at 88.5952 121.92 0)
 			(effects
@@
 			)
 		)
-		(property "Footprint" ""
+		(property "Footprint" "Diode_SMD:D_SOD-123F"
 			(at 111.76 115.57 0)
 			(effects
@@
 		(property "Sim.Pins" "1=K 2=A"
 			(at 111.76 115.57 0)
+			(effects
+				(font
+					(size 1.27 1.27)
+				)
+				(hide yes)
+			)
+		)
+		(property "LCSC" "C64898"
+			(at 111.76 115.57 90)
 			(effects
 				(font
@@
 			)
 		)
-		(property "Footprint" ""
+		(property "Footprint" "Capacitor_THT:CP_Radial_D12.5mm_P5.00mm"
 			(at 96.2152 71.12 0)
 			(effects

Commit message: big ol update
Parts:
- added D7: LED, LED_SMD:LED_0603_1608Metric, symbol Device:LED
- added D9: 5v Zener, Diode_SMD:D_SMA, symbol Device:D
- added F1: 5v Polyfuse, RKEF300:FUS_RKEF300_TYCO_TYC, symbol Device:Polyfuse
- added R11: 1k, Resistor_SMD:R_0805_2012Metric, symbol Device:R
Connections:
- net +5V: now also D9.1 (K), F1.1, R11.2; no longer C2.1, L1.2, U2.4 (FEEDBACK)
- net GND: now also D7.1 (K), D9.2 (A)
- new net: C2.1, F1.2, L1.2, U2.4 (FEEDBACK)
- new net: D7.2 (A), R11.1
