File: PCB/BeanBike/Controller/beanbike_controller_connectors.kicad_sch (KiCad schematic)
At the start: 11 parts, among them J2 Motor Conn, J3 Throttle Conn, J4 PAS Conn, J5 Display Conn, J6 Brake Conn

Commit message: Forgot to commit
Parts:
- J2: footprint Connector_PinHeader_2.54mm:PinHeader_1x08_P2.54mm_Vertical -> (none)
- J3, J4: footprint Connector_PinHeader_2.54mm:PinHeader_1x03_P2.54mm_Vertical -> (none)
- J5: footprint Connector_PinHeader_2.54mm:PinHeader_1x06_P2.54mm_Vertical -> (none)
- J6: footprint Connector_PinHeader_2.54mm:PinHeader_1x02_P2.54mm_Vertical -> (none)
- R10, R11, R6, R7, R8, R9: footprint Resistor_SMD:R_0603_1608Metric -> (none)
Changed lines of the file:
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@@
 		(title "BeanBike Controller Connectors")
 		(date "2025-10-10")
-		(rev "1")
+		(rev "3")
 		(company "Ginobeano")
 	)
@@
 			)
 		)
-		(property "Footprint" "Resistor_SMD:R_0603_1608Metric"
+		(property "Footprint" ""
 			(at 212.598 27.94 90)
 			(effects
@@
 			)
 		)
-		(property "Footprint" "Resistor_SMD:R_0603_1608Metric"
+		(property "Footprint" ""
 			(at 211.328 48.26 90)
 			(effects
@@
 			)
 		)
-		(property "Footprint" "Resistor_SMD:R_0603_1608Metric"
+		(property "Footprint" ""
 			(at 199.39 53.848 90)
 			(effects
@@
 			)
 		)
-		(property "Footprint" "Resistor_SMD:R_0603_1608Metric"
+		(property "Footprint" ""
 			(at 200.66 33.528 90)
 			(effects
@@
 			)
 		)
-		(property "Footprint" "Connector_PinHeader_2.54mm:PinHeader_1x08_P2.54mm_Vertical"
+		(property "Footprint" ""
 			(at 54.61 139.7 0)
 			(effects
@@
 			)
 		)
-		(property "Footprint" "Connector_PinHeader_2.54mm:PinHeader_1x03_P2.54mm_Vertical"
+		(property "Footprint" ""
 			(at 121.92 139.7 0)
 			(effects
@@
 			)
 		)
-		(property "Footprint" "Connector_PinHeader_2.54mm:PinHeader_1x03_P2.54mm_Vertical"
+		(property "Footprint" ""
 			(at 92.71 139.7 0)
 			(effects
@@
 			)
 		)
-		(property "Footprint" "Connector_PinHeader_2.54mm:PinHeader_1x02_P2.54mm_Vertical"
+		(property "Footprint" ""
 			(at 186.69 139.7 0)
 			(effects
@@
 			)
 		)
-		(property "Footprint" "Resistor_SMD:R_0603_1608Metric"
+		(property "Footprint" ""
 			(at 199.39 71.628 90)
 			(effects
@@
 			)
 		)
-		(property "Footprint" "Resistor_SMD:R_0603_1608Metric"
+		(property "Footprint" ""
 			(at 211.328 66.04 90)
 			(effects
@@
 			)
 		)
-		(property "Footprint" "Connector_PinHeader_2.54mm:PinHeader_1x06_P2.54mm_Vertical"
+		(property "Footprint" ""
 			(at 156.21 139.7 0)
 			(effects

Commit message: STM32
Parts:
- added J7: DEBUG Conn, symbol Connector:Conn_01x03_Pin
Connections:
- net GND: now also J7.3 (Pin_3)
- new net MCU_RX: J7.2 (Pin_2)
- new net MCU_TX: J7.1 (Pin_1)
Other:
- note added: "Debug Connector"
Changed lines of the file:
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@@
+	)
+	(rectangle
+		(start 203.2 114.3)
+		(end 233.68 147.32)
+		(stroke
+			(width 0)
+			(type default)
+		)
+		(fill
+			(type none)
+		)
 	)
 	(rectangle
@@
 		(fill
 			(type none)
+		)
+	)
+	(text "Debug Connector\n"
+		(exclude_from_sim no)
+		(at 218.694 113.792 0)
+		(effects
+			(font
+				(size 1.27 1.27)
+			)
 		)
 	)
@@
 	(wire
 		(pts
+			(xy 219.71 128.27) (xy 219.71 134.62)
+		)
+		(stroke
+			(width 0)
+			(type default)
+		)
+	)
+	(wire
+		(pts
 			(xy 209.55 69.85) (xy 223.52 69.85)
 		)
@@
 	(wire
 		(pts
+			(xy 228.6 128.27) (xy 219.71 128.27)
+		)
+		(stroke
+			(width 0)
+			(type default)
+		)
+	)
+	(wire
+		(pts
 			(xy 209.55 52.07) (xy 223.52 52.07)
 		)
@@
 	(wire
 		(pts
+			(xy 214.63 128.27) (xy 214.63 134.62)
+		)
+		(stroke
+			(width 0)
+			(type default)
+		)
+	)
+	(wire
+		(pts
+			(xy 217.17 128.27) (xy 217.17 134.62)
+		)
+		(stroke
+			(width 0)
+			(type default)
+		)
+	)
+	(wire
+		(pts
 			(xy 184.15 52.07) (xy 195.58 52.07)
 		)
@@
 		)
 	)
+	(global_label "MCU_TX"
+		(shape input)
+		(at 214.63 128.27 90)
+		(fields_autoplaced yes)
+		(effects
+			(font
+				(size 1.27 1.27)
+			)
+			(justify left)
+		)
+		(property "Intersheetrefs" "${INTERSHEET_REFS}"
+			(at 214.63 118.0882 90)
+			(effects
+				(font
+					(size 1.27 1.27)
+				)
+				(justify left)
+				(hide yes)
+			)
+		)
+	)
 	(global_label "THROTTLE_DATA"
 		(shape input)
@@
 		(property "Intersheetrefs" "${INTERSHEET_REFS}"
 			(at 124.46 121.112 90)
+			(effects
+				(font
+					(size 1.27 1.27)
+				)
+				(justify left)
+				(hide yes)
+			)
+		)
+	)
+	(global_label "MCU_RX"
+		(shape input)
+		(at 217.17 128.27 90)
+		(fields_autoplaced yes)
+		(effects
+			(font
+				(size 1.27 1.27)
+			)
+			(justify left)
+		)
+		(property "Intersheetrefs" "${INTERSHEET_REFS}"
+			(at 217.17 117.7858 90)
 			(effects
 				(font
@@
 	)
 	(symbol
+		(lib_id "power:GND")
+		(at 228.6 128.27 0)
+		(unit 1)
+		(exclude_from_sim no)
+		(in_bom yes)
+		(on_board yes)
+		(dnp no)
+		(fields_autoplaced yes)
+		(property "Reference" "#PWR038"
+			(at 228.6 134.62 0)
+			(effects
+				(font
+					(size 1.27 1.27)
+				)
+				(hide yes)
+			)
+		)
+		(property "Value" "GND"
+			(at 228.6 133.35 0)
+			(effects
+				(font
+					(size 1.27 1.27)
+				)
+			)
+		)
+		(property "Footprint" ""
+			(at 228.6 128.27 0)
+			(effects
+				(font
+					(size 1.27 1.27)
+				)
+				(hide yes)
+			)
+		)
+		(property "Datasheet" ""
+			(at 228.6 128.27 0)
+			(effects
+				(font
+					(size 1.27 1.27)
+				)
+				(hide yes)
+			)
+		)
+		(property "Description" "Power symbol creates a global label with name \"GND\" , ground"
+			(at 228.6 128.27 0)
+			(effects
+				(font
+					(size 1.27 1.27)
+				)
+				(hide yes)
+			)
+		)
+		(pin "1"
+		)
+		(instances
+			(project ""
+				(path "/645e8d68-d9e1-48b3-98a5-3b81aa58d1ea/2c1bff84-81c5-435a-a8af-2b7800a2d1fe"
+					(reference "#PWR038")
+					(unit 1)
+				)
+			)
+		)
+	)
+	(symbol
 		(lib_id "Device:R")
 		(at 209.55 48.26 180)
@@
 					(unit 1)
 				)
+			)
+		)
+	)
+	(symbol
+		(lib_id "Connector:Conn_01x03_Pin")
+		(at 217.17 139.7 90)
+		(unit 1)
+		(exclude_from_sim no)
+		(in_bom yes)
+		(on_board yes)
+		(dnp no)
+		(fields_autoplaced yes)
+		(property "Reference" "J7"
+			(at 217.17 142.24 90)
+			(effects
+				(font
+					(size 1.27 1.27)
+				)
+			)
+		)
+		(property "Value" "DEBUG Conn"
+			(at 217.17 144.78 90)
+			(effects
+				(font
+					(size 1.27 1.27)
+				)
+			)
+		)
+		(property "Footprint" ""
+			(at 217.17 139.7 0)
+			(effects
+				(font
+					(size 1.27 1.27)
+				)
+				(hide yes)
+			)
+		)
+		(property "Datasheet" "~"
+			(at 217.17 139.7 0)
+			(effects
+				(font
+					(size 1.27 1.27)
+				)
+				(hide yes)
+			)
+		)
+		(property "Description" "Generic connector, single row, 01x03, script generated"
+			(at 217.17 139.7 0)
+			(effects
+				(font
+					(size 1.27 1.27)
+				)
+				(hide yes)
+			)
+		)
+		(pin "1"
+		)
+		(pin "2"
+		)
+		(pin "3"
+		)
+		(instances
+			(project ""
+				(path "/645e8d68-d9e1-48b3-98a5-3b81aa58d1ea/2c1bff84-81c5-435a-a8af-2b7800a2d1fe"
+					(reference "J7")
+					(unit 1)
+				)

Commit message: Footprints
Parts:
- J2: footprint (none) -> Connector_PinHeader_2.54mm:PinHeader_1x08_P2.54mm_Vertical
- J3, J4, J7: footprint (none) -> Connector_PinHeader_2.54mm:PinHeader_1x03_P2.54mm_Vertical
- J5: footprint (none) -> Connector_PinHeader_2.54mm:PinHeader_1x06_P2.54mm_Vertical
- J6: footprint (none) -> Connector_PinHeader_2.54mm:PinHeader_1x02_P2.54mm_Vertical
- R10, R6, R8: footprint (none) -> Resistor_SMD:R_0805_2012Metric; LCSC C98220 -> C17414
- R11, R7, R9: footprint (none) -> Resistor_SMD:R_0805_2012Metric; LCSC C137655 -> C17506
Changed lines of the file:
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@@
 			)
 		)
-		(property "Footprint" ""
+		(property "Footprint" "Resistor_SMD:R_0805_2012Metric"
 			(at 212.598 27.94 90)
 			(effects
@@
 			)
 		)
-		(property "LCSC" "C137655"
+		(property "LCSC" "C17506"
 			(at 210.82 27.94 0)
 			(effects
@@
 			)
 		)
-		(property "Footprint" ""
+		(property "Footprint" "Resistor_SMD:R_0805_2012Metric"
 			(at 211.328 48.26 90)
 			(effects
@@
 			)
 		)
-		(property "LCSC" "C137655"
+		(property "LCSC" "C17506"
 			(at 209.55 48.26 0)
 			(effects
@@
 			)
 		)
-		(property "Footprint" ""
+		(property "Footprint" "Resistor_SMD:R_0805_2012Metric"
 			(at 199.39 53.848 90)
 			(effects
@@
 			)
 		)
-		(property "LCSC" "C98220"
+		(property "LCSC" "C17414"
 			(at 199.39 52.07 90)
 			(effects
@@
 			)
 		)
-		(property "Footprint" ""
+		(property "Footprint" "Resistor_SMD:R_0805_2012Metric"
 			(at 200.66 33.528 90)
 			(effects
@@
 			)
 		)
-		(property "LCSC" "C98220"
+		(property "LCSC" "C17414"
 			(at 200.66 31.75 90)
 			(effects
@@
 			)
 		)
-		(property "Footprint" ""
+		(property "Footprint" "Connector_PinHeader_2.54mm:PinHeader_1x08_P2.54mm_Vertical"
 			(at 54.61 139.7 0)
 			(effects
@@
 			)
 		)
-		(property "Footprint" ""
+		(property "Footprint" "Connector_PinHeader_2.54mm:PinHeader_1x03_P2.54mm_Vertical"
 			(at 121.92 139.7 0)
 			(effects
@@
 			)
 		)
-		(property "Footprint" ""
+		(property "Footprint" "Connector_PinHeader_2.54mm:PinHeader_1x03_P2.54mm_Vertical"
 			(at 92.71 139.7 0)
 			(effects
@@
 			)
 		)
-		(property "Footprint" ""
+		(property "Footprint" "Connector_PinHeader_2.54mm:PinHeader_1x02_P2.54mm_Vertical"
 			(at 186.69 139.7 0)
 			(effects
@@
 			)
 		)
-		(property "Footprint" ""
+		(property "Footprint" "Resistor_SMD:R_0805_2012Metric"
 			(at 199.39 71.628 90)
 			(effects
@@
 			)
 		)
-		(property "LCSC" "C98220"
+		(property "LCSC" "C17414"
 			(at 199.39 69.85 90)
 			(effects
@@
 			)
 		)
-		(property "Footprint" ""
+		(property "Footprint" "Resistor_SMD:R_0805_2012Metric"
 			(at 211.328 66.04 90)
 			(effects
@@
 			)
 		)
-		(property "LCSC" "C137655"
+		(property "LCSC" "C17506"
 			(at 209.55 66.04 0)
 			(effects
@@
 			)
 		)
-		(property "Footprint" ""
+		(property "Footprint" "Connector_PinHeader_2.54mm:PinHeader_1x06_P2.54mm_Vertical"
 			(at 156.21 139.7 0)
 			(effects
@@
 			)
 		)
-		(property "Footprint" ""
+		(property "Footprint" "Connector_PinHeader_2.54mm:PinHeader_1x03_P2.54mm_Vertical"
 			(at 217.17 139.7 0)
 			(effects

Commit message: PCB v3
Parts:
- removed R10, R6, R8: 10k, Resistor_SMD:R_0805_2012Metric, symbol Device:R
- removed R11, R7, R9: 18k, Resistor_SMD:R_0805_2012Metric, symbol Device:R
- added U6: SN74LVC4245APWR, easyeda2kicad:TSSOP-24_L7.8-W4.4-P0.65-LS6.4-BL, symbol easyeda2kicad:SN74LVC4245APWR
Connections:
- net +5V: now also U6.1 (VCCA), U6.2 (DIR)
- net GND: now also U6.11 (GND), U6.12 (GND), U6.13 (GND), U6.22 (~{OE})
- net MOTOR_HALL_A: now also U6.3 (A1)
- net MOTOR_HALL_B: now also U6.4 (A2)
- net MOTOR_HALL_C: now also U6.5 (A3)
- net MCU-Boot renamed BOOT
- net MCU-GPIO34 renamed THROTTLE_DATA
- net THROTTLE_DATA: now also U6.6 (A4)
- net MCU-GPIO35 renamed PAS_PULSE
- net PAS_PULSE: now also U6.7 (A5)
- net MCU-RX renamed MCU_CAN+
- net MCU-Reset renamed RST
- net MCU-TX renamed MCU_CAN-
- new net +3.3V: U6.23 (VCCB), U6.24 (VCCB)
- new net MCU_PB0: U6.18 (B4)
- new net MCU_PB1: U6.17 (B5)
- new net MCU_PB2: U6.21 (B1)
- new net MCU_PB3: U6.20 (B2)
- new net MCU_PB4: U6.19 (B3)
- no-connect marks 0 -> 6

Commit message: PCB v3
Parts:
- removed J2: Motor Conn, Connector_PinHeader_2.54mm:PinHeader_1x08_P2.54mm_Vertical, symbol Connector:Conn_01x08_Pin
- added J10: PHASE C, 8196:KEYSTONE_8196, symbol 8196:8196
- added J2: Conn_01x05_Pin, Connector_PinHeader_2.54mm:PinHeader_1x05_P2.54mm_Vertical, symbol Connector:Conn_01x05_Pin
- added J8: PHASE A, 8196:KEYSTONE_8196, symbol 8196:8196
- added J9: PHASE B, 8196:KEYSTONE_8196, symbol 8196:8196
Connections:
- net +5V: now also J2.1 (Pin_1)
- net GND: now also J2.2 (Pin_2)
- net MOTOR_HALL_A: now also J2.3 (Pin_3)
- net MOTOR_HALL_B: now also J2.4 (Pin_4)
- net MOTOR_HALL_C: now also J2.5 (Pin_5)
- net MOTOR_PHASE_A: now also J8.1_1 (1), J8.1_2 (1__1), J8.1_3 (1__2), J8.1_4 (1__3), J8.1_5 (1__4), J8.1_6 (1__5)
- net MOTOR_PHASE_B: now also J9.1_1 (1), J9.1_2 (1__1), J9.1_3 (1__2), J9.1_4 (1__3), J9.1_5 (1__4), J9.1_6 (1__5)
- net MOTOR_PHASE_C: now also J10.1_1 (1), J10.1_2 (1__1), J10.1_3 (1__2), J10.1_4 (1__3), J10.1_5 (1__4), J10.1_6 (1__5)
- net MCU_PB2 renamed MCU_PC0
- net MCU_PB3 renamed MCU_PC1
- net MCU_PB4 renamed MCU_PC2
Other:
- note added: "Motor Encoder Connector"
- note removed: "Motor Connector"

Commit message: big ol update
Parts:
- removed J7: DEBUG Conn, Connector_PinHeader_2.54mm:PinHeader_1x03_P2.54mm_Vertical, symbol Connector:Conn_01x03_Pin
- added J7: ST-Link-Debug, Connector_PinHeader_2.54mm:PinHeader_1x06_P2.54mm_Vertical, symbol Connector:Conn_01x06_Pin
Connections:
- net +3.3V: now also J7.1 (Pin_1)
- net GND: now also J7.6 (Pin_6)
- net RST: now also J7.5 (Pin_5)
- new net MCU_SWCLK: J7.3 (Pin_3)
- new net MCU_SWDIO: J7.2 (Pin_2)
- new net MCU_SWO: J7.4 (Pin_4)
