File: PCB/BeanBike/Controller/beanbike_controller_motor.kicad_sch (KiCad schematic)
At the start: 19 parts, among them Q1 PHASE A HIGH, Q2 PHASE B HIGH, Q3 PHASE C HIGH, Q4 PHASE A LOW, Q5 PHASE B LOW, Q6 PHASE C LOW, U5 DRV8353SRTAT

Commit message: Forgot to commit
Parts:
- C18, C20, C21, C22, C23, C24: footprint Capacitor_SMD:C_0201_0603Metric -> (none)
- C19: footprint Capacitor_SMD:C_0603_1608Metric -> (none)
- Q1, Q2, Q3, Q4, Q5, Q6: footprint Package_TO_SOT_THT:TO-220-3_Vertical -> (none)
- R25, R26: footprint Resistor_SMD:R_0603_1608Metric -> (none)
- R3, R4, R5: footprint Resistor_SMD:R_2512_6332Metric -> (none)
- U5: footprint MOTORIC:RTA0040B -> (none)
Changed lines of the file:
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@@
 		(title "BeanBike Controller Motor")
 		(date "2025-10-11")
-		(rev "1")
+		(rev "3")
 		(company "Ginobeano")
 	)
@@
 			)
 		)
-		(property "Footprint" "Capacitor_SMD:C_0201_0603Metric"
+		(property "Footprint" ""
 			(at 77.47 39.37 0)
 			(effects
@@
 			)
 		)
-		(property "Footprint" "Package_TO_SOT_THT:TO-220-3_Vertical"
+		(property "Footprint" ""
 			(at 252.73 105.41 0)
 			(effects
@@
 			)
 		)
-		(property "Footprint" "MOTORIC:RTA0040B"
+		(property "Footprint" ""
 			(at 109.22 102.87 0)
 			(effects
@@
 			)
 		)
-		(property "Footprint" "Package_TO_SOT_THT:TO-220-3_Vertical"
+		(property "Footprint" ""
 			(at 252.73 138.43 0)
 			(effects
@@
 			)
 		)
-		(property "Footprint" "Package_TO_SOT_THT:TO-220-3_Vertical"
+		(property "Footprint" ""
 			(at 261.62 44.45 0)
 			(effects
@@
 			)
 		)
-		(property "Footprint" "Package_TO_SOT_THT:TO-220-3_Vertical"
+		(property "Footprint" ""
 			(at 261.62 62.23 0)
 			(effects
@@
 			)
 		)
-		(property "Footprint" "Resistor_SMD:R_0603_1608Metric"
+		(property "Footprint" ""
 			(at 82.55 130.81 0)
 			(effects
@@
 			)
 		)
-		(property "Footprint" "Capacitor_SMD:C_0201_0603Metric"
+		(property "Footprint" ""
 			(at 77.47 49.53 0)
 			(effects
@@
 			)
 		)
-		(property "Footprint" "Resistor_SMD:R_2512_6332Metric"
+		(property "Footprint" ""
 			(at 136.652 146.05 90)
 			(effects
@@
 			)
 		)
-		(property "Footprint" "Capacitor_SMD:C_0201_0603Metric"
+		(property "Footprint" ""
 			(at 80.01 67.31 0)
 			(effects
@@
 			)
 		)
-		(property "Footprint" "Resistor_SMD:R_2512_6332Metric"
+		(property "Footprint" ""
 			(at 136.652 115.57 90)
 			(effects
@@
 			)
 		)
-		(property "Footprint" "Capacitor_SMD:C_0201_0603Metric"
+		(property "Footprint" ""
 			(at 84.7852 62.23 0)
 			(effects
@@
 			)
 		)
-		(property "Footprint" "Package_TO_SOT_THT:TO-220-3_Vertical"
+		(property "Footprint" ""
 			(at 252.73 120.65 0)
 			(effects
@@
 			)
 		)
-		(property "Footprint" "Capacitor_SMD:C_0603_1608Metric"
+		(property "Footprint" ""
 			(at 64.77 39.37 0)
 			(effects
@@
 			)
 		)
-		(property "Footprint" "Capacitor_SMD:C_0201_0603Metric"
+		(property "Footprint" ""
 			(at 45.72 140.97 0)
 			(effects
@@
 			)
 		)
-		(property "Footprint" "Package_TO_SOT_THT:TO-220-3_Vertical"
+		(property "Footprint" ""
 			(at 261.62 29.21 0)
 			(effects
@@
 			)
 		)
-		(property "Footprint" "Capacitor_SMD:C_0201_0603Metric"
+		(property "Footprint" ""
 			(at 66.04 125.73 0)
 			(effects
@@
 			)
 		)
-		(property "Footprint" "Resistor_SMD:R_0603_1608Metric"
+		(property "Footprint" ""
 			(at 44.958 101.6 90)
 			(effects
@@
 			)
 		)
-		(property "Footprint" "Resistor_SMD:R_2512_6332Metric"
+		(property "Footprint" ""
 			(at 136.652 130.81 90)
 			(effects

Commit message: Schematic v3 Done
Connections:
- net VDRAIN is gone; now on net PWR_MOTOR: C20.2, U5.4 (VDRAIN)
- net GND: no longer Q4.2 (D), Q5.2 (D), Q6.2 (D)
- net MOTOR_PHASE_A: now also Q4.2 (D); no longer Q4.3 (S), R5.1, U5.9 (SPA)
- net MOTOR_PHASE_B: now also Q5.2 (D); no longer Q5.3 (S), R4.1, U5.12 (SPB)
- net MOTOR_PHASE_C: now also Q6.2 (D); no longer Q6.3 (S), R3.1, U5.19 (SPC)
- net MCU-GPIO12 renamed MCU_INHA
- net MCU-GPIO13 renamed MCU_PC9
- net MCU-GPIO14 renamed MCU_INLA
- net MCU-GPIO15 renamed MCU_PC8
- net MCU-GPIO17 renamed MCU_SOC
- net MCU-GPIO18 renamed MCU_SPI1_SCK
- net MCU-GPIO19 renamed MCU_SPI1_MOSI
- net MCU-GPIO21 renamed MCU_SOA
- net MCU-GPIO22 renamed MCU_SOB
- net MCU-GPIO23 renamed MCU_SPI1_MISO
- net MCU-GPIO25 renamed MCU_INHC
- net MCU-GPIO26 renamed MCU_INLB
- net MCU-GPIO27 renamed MCU_INHB
- net MCU-GPIO33 renamed MCU_INLC
- net MCU-GPIO5 renamed MCU_PA4
- new net: Q4.3 (S), R5.1, U5.9 (SPA)
- new net: Q5.3 (S), R4.1, U5.12 (SPB)
- new net: Q6.3 (S), R3.1, U5.19 (SPC)
Other:
- moved on the sheet: Q4, Q6

Commit message: Footprints
Parts:
- C18, C24: footprint (none) -> Capacitor_SMD:C_0402_1005Metric; LCSC C335106 -> C1525
- C19: footprint (none) -> Capacitor_SMD:C_0805_2012Metric; LCSC C84419 -> C45783
- C20, C22, C23: footprint (none) -> Capacitor_SMD:C_0402_1005Metric; LCSC C87144 -> C52923
- C21: footprint (none) -> Capacitor_SMD:C_0603_1608Metric; LCSC C88917 -> C1622
- Q1, Q2, Q3, Q4, Q5, Q6: footprint (none) -> TO-220AB:TO254P1050X476X2020-3
- R25, R26: footprint (none) -> Resistor_SMD:R_0805_2012Metric; LCSC C163420 -> C17819
- R3, R4, R5: footprint (none) -> footprints:RES_1L00x_BRN
- U5: footprint (none) -> DRV8353:QFN50P600X600X80-41N
Changed lines of the file:
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@@
 			)
 		)
-		(property "Footprint" ""
+		(property "Footprint" "Capacitor_SMD:C_0402_1005Metric"
 			(at 77.47 39.37 0)
 			(effects
@@
 			)
 		)
-		(property "LCSC" "C335106"
+		(property "LCSC" "C1525"
 			(at 77.47 39.37 0)
 			(effects
@@
 			)
 		)
-		(property "Footprint" ""
+		(property "Footprint" "TO-220AB:TO254P1050X476X2020-3"
 			(at 252.73 138.43 0)
 			(effects
@@
 			)
 		)
-		(property "Footprint" ""
+		(property "Footprint" "DRV8353:QFN50P600X600X80-41N"
 			(at 109.22 102.87 0)
 			(effects
@@
 			)
 		)
-		(property "Footprint" ""
+		(property "Footprint" "TO-220AB:TO254P1050X476X2020-3"
 			(at 252.73 101.6 0)
 			(effects
@@
 			)
 		)
-		(property "Footprint" ""
+		(property "Footprint" "TO-220AB:TO254P1050X476X2020-3"
 			(at 261.62 44.45 0)
 			(effects
@@
 			)
 		)
-		(property "Footprint" ""
+		(property "Footprint" "TO-220AB:TO254P1050X476X2020-3"
 			(at 261.62 62.23 0)
 			(effects
@@
 			)
 		)
-		(property "Footprint" ""
+		(property "Footprint" "Resistor_SMD:R_0805_2012Metric"
 			(at 82.55 130.81 0)
 			(effects
@@
 			)
 		)
-		(property "LCSC" "C163420"
+		(property "LCSC" "C17819"
 			(at 82.55 130.81 0)
 			(effects
@@
 			)
 		)
-		(property "Footprint" ""
+		(property "Footprint" "Capacitor_SMD:C_0402_1005Metric"
 			(at 77.47 49.53 0)
 			(effects
@@
 			)
 		)
-		(property "LCSC" "C87144"
+		(property "LCSC" "C52923"
 			(at 77.47 49.53 0)
 			(effects
@@
 			)
 		)
-		(property "Footprint" ""
+		(property "Footprint" "footprints:RES_1L00x_BRN"
 			(at 136.652 146.05 90)
 			(effects
@@
 			)
 		)
-		(property "Footprint" ""
+		(property "Footprint" "Capacitor_SMD:C_0402_1005Metric"
 			(at 80.01 67.31 0)
 			(effects
@@
 			)
 		)
-		(property "LCSC" "C87144"
+		(property "LCSC" "C52923"
 			(at 80.01 67.31 0)
 			(effects
@@
 			)
 		)
-		(property "Footprint" ""
+		(property "Footprint" "footprints:RES_1L00x_BRN"
 			(at 136.652 115.57 90)
 			(effects
@@
 			)
 		)
-		(property "Footprint" ""
+		(property "Footprint" "Capacitor_SMD:C_0603_1608Metric"
 			(at 84.7852 62.23 0)
 			(effects
@@
 			)
 		)
-		(property "LCSC" "C88917"
+		(property "LCSC" "C1622"
 			(at 83.82 58.42 0)
 			(effects
@@
 			)
 		)
-		(property "Footprint" ""
+		(property "Footprint" "TO-220AB:TO254P1050X476X2020-3"
 			(at 252.73 120.65 0)
 			(effects
@@
 			)
 		)
-		(property "Footprint" ""
+		(property "Footprint" "Capacitor_SMD:C_0805_2012Metric"
 			(at 64.77 39.37 0)
 			(effects
@@
 			)
 		)
-		(property "LCSC" "C84419"
+		(property "LCSC" "C45783"
 			(at 64.77 39.37 0)
 			(effects
@@
 			)
 		)
-		(property "Footprint" ""
+		(property "Footprint" "Capacitor_SMD:C_0402_1005Metric"
 			(at 45.72 140.97 0)
 			(effects
@@
 			)
 		)
-		(property "LCSC" "C335106"
+		(property "LCSC" "C1525"
 			(at 45.72 140.97 0)
 			(effects
@@
 			)
 		)
-		(property "Footprint" ""
+		(property "Footprint" "TO-220AB:TO254P1050X476X2020-3"
 			(at 261.62 29.21 0)
 			(effects
@@
 			)
 		)
-		(property "Footprint" ""
+		(property "Footprint" "Capacitor_SMD:C_0402_1005Metric"
 			(at 66.04 125.73 0)
 			(effects
@@
 			)
 		)
-		(property "LCSC" "C87144"
+		(property "LCSC" "C52923"
 			(at 66.04 125.73 0)
 			(effects
@@
 			)
 		)
-		(property "Footprint" ""
+		(property "Footprint" "Resistor_SMD:R_0805_2012Metric"
 			(at 44.958 101.6 90)
 			(effects
@@
 			)
 		)
-		(property "LCSC" "C163420"
+		(property "LCSC" "C17819"
 			(at 43.18 101.6 0)
 			(effects
@@
 			)
 		)
-		(property "Footprint" ""
+		(property "Footprint" "footprints:RES_1L00x_BRN"
 			(at 136.652 130.81 90)
 			(effects

Commit message: PCB v3
Other:
- moved on the sheet: R26
Changed lines of the file:
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@@
 	)
 	(junction
-		(at 82.55 133.35)
+		(at 80.01 133.35)
 		(diameter 0)
 		(color 0 0 0 0)
@@
 	(wire
 		(pts
-			(xy 77.47 133.35) (xy 82.55 133.35)
+			(xy 77.47 133.35) (xy 80.01 133.35)
 		)
 		(stroke
@@
 	(wire
 		(pts
-			(xy 82.55 133.35) (xy 86.36 133.35)
-		)
-		(stroke
-			(width 0)
-			(type default)
-		)
-	)
-	(wire
-		(pts
 			(xy 83.82 54.61) (xy 86.36 54.61)
 		)
@@
 	(wire
 		(pts
+			(xy 80.01 133.35) (xy 86.36 133.35)
+		)
+		(stroke
+			(width 0)
+			(type default)
+		)
+	)
+	(wire
+		(pts
 			(xy 77.47 46.99) (xy 86.36 46.99)
 		)
@@
 	(wire
 		(pts
-			(xy 82.55 127) (xy 82.55 128.27)
+			(xy 80.01 127) (xy 80.01 128.27)
 		)
 		(stroke
@@
 		(pts
 			(xy 67.31 97.79) (xy 86.36 97.79)
+		)
+		(stroke
+			(width 0)
+			(type default)
+		)
+	)
+	(wire
+		(pts
+			(xy 80.01 127) (xy 82.55 127)
 		)
 		(stroke
@@
 	(symbol
 		(lib_id "Device:R_Small")
-		(at 82.55 130.81 0)
+		(at 80.01 130.81 0)
 		(unit 1)
 		(exclude_from_sim no)
@@
 		(fields_autoplaced yes)
 		(property "Reference" "R26"
-			(at 85.09 129.5399 0)
+			(at 82.55 129.5399 0)
 			(effects
 				(font
@@
 		)
 		(property "Value" "73k"
-			(at 85.09 132.0799 0)
+			(at 82.55 132.0799 0)
 			(effects
 				(font
@@
 		)
 		(property "Footprint" "Resistor_SMD:R_0805_2012Metric"
-			(at 82.55 130.81 0)
+			(at 80.01 130.81 0)
 			(effects
 				(font
@@
 		)
 		(property "Datasheet" "~"
-			(at 82.55 130.81 0)
+			(at 80.01 130.81 0)
 			(effects
 				(font
@@
 		)
 		(property "Description" "Resistor, small symbol"
-			(at 82.55 130.81 0)
+			(at 80.01 130.81 0)
 			(effects
 				(font
@@
 		)
 		(property "LCSC" "C17819"
-			(at 82.55 130.81 0)
-			(effects
-				(font
+			(at 80.01 130.81 0)
+			(effects
+				(font

Commit message: big ol update
Parts:
- added D4, D5, D6: LED, LED_SMD:LED_0603_1608Metric, symbol Device:LED
- added R10, R8, R9: 15k, Resistor_SMD:R_0805_2012Metric, symbol Device:R
Connections:
- net GND: now also D4.1 (K), D5.1 (K), D6.1 (K)
- net MOTOR_PHASE_A: now also R8.2
- net MOTOR_PHASE_B: now also R9.2
- net MOTOR_PHASE_C: now also R10.2
- net PWR_MOTOR: now also C18.1, C19.1, U5.3 (VM)
- new net: D6.2 (A), R10.1
- new net: D5.2 (A), R9.1
- new net: D4.2 (A), R8.1
