File: PCB/BeanBike/Controller/beanbike_power.kicad_sch (KiCad schematic)
At the start: 4 parts, among them J1 XT80 Male

Commit message: Forgot to commit
Parts:
- F1: footprint Fuse:Fuse_1206_3216Metric -> (none)
- J1: footprint Connector_Wire:SolderWire-2sqmm_1x02_P7.8mm_D2mm_OD3.9mm -> (none)
- R1, R2: footprint Resistor_SMD:R_0603_1608Metric -> (none)
Changed lines of the file:
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@@
 	(title_block
 		(title "BeanBike Controller Power")
-		(rev "1")
+		(rev "3")
 		(company "Ginobeano")
 	)
@@
 			)
 		)
-		(property "Footprint" "Resistor_SMD:R_0603_1608Metric"
+		(property "Footprint" ""
 			(at 35.052 125.73 90)
 			(effects
@@
 			)
 		)
-		(property "Footprint" "Connector_Wire:SolderWire-2sqmm_1x02_P7.8mm_D2mm_OD3.9mm"
+		(property "Footprint" ""
 			(at 19.05 59.69 0)
 			(effects
@@
 			)
 		)
-		(property "Footprint" "Resistor_SMD:R_0603_1608Metric"
+		(property "Footprint" ""
 			(at 43.942 125.73 90)
 			(effects
@@
 			)
 		)
-		(property "Footprint" "Fuse:Fuse_1206_3216Metric"
+		(property "Footprint" ""
 			(at 26.67 85.598 90)
 			(effects

Commit message: STM32
Parts:
- removed F1: Fuse, symbol Device:Fuse
Connections:
- net PWR_MOTOR is gone; now on net +BATT: R2.1
Changed lines of the file:
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@@
 	(wire
 		(pts
-			(xy 30.48 83.82) (xy 46.99 83.82)
+			(xy 22.86 83.82) (xy 46.99 83.82)
 		)
 		(stroke
@@
 					(unit 1)
 				)
-			)
-		)
-	)
-	(symbol
-		(lib_id "Device:Fuse")
-		(at 26.67 83.82 90)
-		(unit 1)
-		(exclude_from_sim no)
-		(in_bom yes)
-		(on_board yes)
-		(dnp no)
-		(fields_autoplaced yes)
-		(property "Reference" "F1"
-			(at 26.67 77.47 90)
-			(effects
-				(font
-					(size 1.27 1.27)
-				)
-			)
-		)
-		(property "Value" "Fuse"
-			(at 26.67 80.01 90)
-			(effects
-				(font
-					(size 1.27 1.27)
-				)
-			)
-		)
-		(property "Footprint" ""
-			(at 26.67 85.598 90)
-			(effects
-				(font
-					(size 1.27 1.27)
-				)
-				(hide yes)
-			)
-		)
-		(property "Datasheet" "~"
-			(at 26.67 83.82 0)
-			(effects
-				(font
-					(size 1.27 1.27)
-				)
-				(hide yes)
-			)
-		)
-		(property "Description" "Fuse"
-			(at 26.67 83.82 0)
-			(effects
-				(font
-					(size 1.27 1.27)
-				)
-				(hide yes)
-			)
-		)
-		(property "LCSC" "C22445177"
-			(at 26.67 83.82 90)
-			(effects
-				(font
-					(size 1.27 1.27)
-				)
-				(hide yes)
-			)
-		)
-		(pin "1"
-		)
-		(pin "2"
-		)
-		(instances
-			(project ""
-				(path "/645e8d68-d9e1-48b3-98a5-3b81aa58d1ea/ceef88aa-c829-4630-8455-6c437ac60286"
-					(reference "F1")
-					(unit 1)
-				)

Commit message: Schematic v3 Done
Changed lines of the file:
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@@
+	(wire
+		(pts
+			(xy 24.13 59.69) (xy 34.29 59.69)
+		)
+		(stroke
+			(width 0)
+			(type default)
+		)
+	)
+	(wire
+		(pts
+			(xy 24.13 62.23) (xy 35.56 62.23)
+		)
+		(stroke
+			(width 0)
+			(type default)
+		)
+	)
 	(wire
 		(pts
@@
 	(symbol
 		(lib_id "power:+BATT")
-		(at 24.13 59.69 270)
+		(at 34.29 59.69 270)
 		(unit 1)
 		(exclude_from_sim no)
@@
 		(fields_autoplaced yes)
 		(property "Reference" "#PWR02"
-			(at 20.32 59.69 0)
+			(at 30.48 59.69 0)
 			(effects
 				(font
@@
 		)
 		(property "Value" "+BATT"
-			(at 27.94 59.6899 90)
-			(effects
-				(font
-					(size 1.27 1.27)
-				)
-				(justify left)
-			)
-		)
-		(property "Footprint" ""
-			(at 24.13 59.69 0)
+			(at 38.1 59.6899 90)
+			(effects
+				(font
+					(size 1.27 1.27)
+				)
+				(justify left)
+			)
+		)
+		(property "Footprint" ""
+			(at 34.29 59.69 0)
 			(effects
 				(font
@@
 		)
 		(property "Datasheet" ""
-			(at 24.13 59.69 0)
+			(at 34.29 59.69 0)
 			(effects
 				(font
@@
 		)
 		(property "Description" "Power symbol creates a global label with name \"+BATT\""
-			(at 24.13 59.69 0)
+			(at 34.29 59.69 0)
 			(effects
 				(font
@@
 	(symbol
 		(lib_id "power:GND")
-		(at 24.13 62.23 0)
+		(at 35.56 62.23 0)
 		(unit 1)
 		(exclude_from_sim no)
@@
 		(fields_autoplaced yes)
 		(property "Reference" "#PWR03"
-			(at 24.13 68.58 0)
+			(at 35.56 68.58 0)
 			(effects
 				(font
@@
 		)
 		(property "Value" "GND"
-			(at 24.13 67.31 0)
-			(effects
-				(font
-					(size 1.27 1.27)
-				)
-			)
-		)
-		(property "Footprint" ""
-			(at 24.13 62.23 0)
+			(at 35.56 67.31 0)
+			(effects
+				(font
+					(size 1.27 1.27)
+				)
+			)
+		)
+		(property "Footprint" ""
+			(at 35.56 62.23 0)
 			(effects
 				(font
@@
 		)
 		(property "Datasheet" ""
-			(at 24.13 62.23 0)
+			(at 35.56 62.23 0)
 			(effects
 				(font
@@
 		)
 		(property "Description" "Power symbol creates a global label with name \"GND\" , ground"
-			(at 24.13 62.23 0)
-			(effects
-				(font
+			(at 35.56 62.23 0)
+			(effects
+				(font

Commit message: Footprints
Parts:
- J1: footprint (none) -> XT60PW-M:AMASS_XT60PW-M
- R1: footprint (none) -> Resistor_SMD:R_0805_2012Metric; LCSC C98220 -> C17414
- R2: footprint (none) -> Resistor_SMD:R_0805_2012Metric; LCSC C137657 -> C17501
Changed lines of the file:
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@@
 			)
 		)
-		(property "Footprint" ""
+		(property "Footprint" "Resistor_SMD:R_0805_2012Metric"
 			(at 35.052 125.73 90)
 			(effects
@@
 			)
 		)
-		(property "LCSC" "C98220"
+		(property "LCSC" "C17414"
 			(at 36.83 125.73 0)
 			(effects
@@
 			)
 		)
-		(property "Footprint" ""
+		(property "Footprint" "XT60PW-M:AMASS_XT60PW-M"
 			(at 19.05 59.69 0)
 			(effects
@@
 			)
 		)
-		(property "Footprint" ""
+		(property "Footprint" "Resistor_SMD:R_0805_2012Metric"
 			(at 43.942 125.73 90)
 			(effects
@@
 			)
 		)
-		(property "LCSC" "C137657"
+		(property "LCSC" "C17501"
 			(at 45.72 125.73 0)
 			(effects

Commit message: big ol update
Parts:
- removed J1: XT80 Male, XT60PW-M:AMASS_XT60PW-M, symbol Connector:Conn_01x02_Pin
- added D2: LED, LED_SMD:LED_0603_1608Metric, symbol Device:LED
- added J1: XT60 +, MountingHole:MountingHole_3.2mm_M3_Pad_Via, symbol Connector:Conn_01x01_Pin
- added J11: XT60 -, MountingHole:MountingHole_3.2mm_M3_Pad_Via, symbol Connector:Conn_01x01_Pin
- added R6: 15k, Resistor_SMD:R_0805_2012Metric, symbol Device:R
Connections:
- net +BATT: now also J1.1 (Pin_1), R6.2
- net GND: now also D2.1 (K), J11.1 (Pin_1)
- new net: D2.2 (A), R6.1
